File: hardware/hardware.kicad_sch (KiCad schematic)
At the start: 23 parts, among them IC1 TP5000-QFN16, J1 LiFePO4 3.2V 6000mah 32700 + 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, J2 Solar panel, J3 BME280 / I²C, J4 CJMCU-3935 / I²C, J6 SMD USB-3.1 Type-C Female 16P, U1 ESP32-C3_SUPERMINI, U2 DS3231SN, U3 FM24CL16B, U4 BME280, U5 E22-900MM22S, U6 CJMCU-3935, U7 MCP6542T-I/MS, U9 TPS631000DRLR

Commit message: hardware draft v2
Parts:
- removed BT1: CR2032, Battery:BatteryHolder_Multicomp_BC-2001_1x2032, symbol Device:Battery_Cell
- removed C1: 22 uF, symbol Device:C_Small
- removed C2: 47 uF, symbol Device:C_Small
- removed C3, C4: 100 nF, symbol Device:C_Small
- removed IC1: TP5000-QFN16, TP5000-QFN16:QFN65P400X400X90-17N-D, symbol TP5000-QFN16:TP5000-QFN16
- removed J1: LiFePO4 3.2V 6000mah 32700 + B57861S0103A039 (NTC), Connector_JST:JST_XH_B3B-XH-A_1x03_P2.50mm_Vertical, symbol Connector_Generic:Conn_01x03
- removed J2: Solar panel, Connector_JST:JST_XH_B2B-XH-A_1x02_P2.50mm_Vertical, symbol Connector_Generic:Conn_01x02
- removed J6: SMD USB-3.1 Type-C Female 16P, Connector_USB:USB_C_Receptacle_G-Switch_GT-USB-7010ASV, symbol Connector:USB_C_Receptacle_USB2.0_16P
- removed L2: IHLP1212BZER1R0M11, IHLP1212BZER1R0M11:IND_IHLP1212BZER1R0M11, symbol IHLP1212BZER1R0M11:IHLP1212BZER1R0M11
- removed R1: 511 kOm, symbol Device:R_Small
- removed R2: 91 kOm, symbol Device:R_Small
- removed U7: MCP6542T-I/MS, MCP6542T-I-MS:MSOP8_MC_MCH, symbol ul_MCP6542T-I-MS:MCP6542T-I_MS
- removed U9: TPS631000DRLR, TPS631000DRLR:TPS631000DRLR_TEX, symbol ul_TPS631000DRLR:TPS631000DRLR
- added IC2, IC3: ${DEVICE}, ICs And Semiconductors SMD:SOP50P490X110-10N, symbol CERN:Analog & Interface/INA226AIDGST
Connections:
- net +3V3: now also J3.1 (Pin_1), J4.1 (Pin_1)
- net GND: now also J3.2 (Pin_2), J4.2 (Pin_2), U1.G (GND)
- no-connect marks 0 -> 1
Other:
- note added: "Контроль заряду акумулятора"
- note added: "Скільки W генерує сонячна панель"
- note removed: "+"
- note removed: "-"
- note removed: "3v3"
- note removed: "DC-DC"
- note removed: "GND"
- note removed: "Power"
- note removed: "Контролер заряду"
- note removed: "Контроль температури акумулятора"

Commit message: hardware: power
Parts:
- added R1: 10k, Resistor_SMD:R_0603_1608Metric, symbol Device:R_Small
- renumbered IC2 to IC1, IC3 to IC2, J3 to J1, J4 to J2, U2 to U1, U1 to U2, U6 to U3, U3 to U4, U4 to U5, U5 to U6
Connections:
- net +3V3: now also R1.2
- new net CHARGE_SOURCE_STATUS_OUT: R1.1
Other:
- moved on the sheet: IC2, U5

Commit message: hardware root
Parts:
- removed J2: CJMCU-3935 / I²C, Connector_JST:JST_PH_B6B-PH-K_1x06_P2.00mm_Vertical, symbol Connector_Generic:Conn_01x06
- added C1, C16, C17, C2: 100nF, Capacitor_SMD:C_0603_1608Metric, symbol Device:C_Small
- added J6: CJMCU-3935, Connector_JST:JST_PH_B4B-PH-K_1x04_P2.00mm_Vertical, symbol Connector_Generic:Conn_01x05
- added R16: R_Small, symbol Device:R_Small
- added R2, R3: 4.7k, Resistor_SMD:R_0603_1608Metric, symbol Device:R_Small
- J1: value BME280 / I²C -> BME280
- renumbered IC2 to IC1, IC1 to IC2
Connections:
- net +3V3: now also IC1.1 (A1), IC1.6 (VS+), IC2.2 (A0), IC2.6 (VS+), U3.1 (A1), U3.11 (VCC), U3.2 (A0), U3.3 (EN_V), U3.5 (SI), U4.8 (VDD), C1.2, C16.2, C17.2, C2.2, J6.1 (Pin_1), R2.2, R3.2
- net CHARGE_SOURCE_STATUS_OUT: now also U2.6 (GPIO6)
- net GND: now also IC1.2 (A0), IC1.7 (GND), IC2.1 (A1), IC2.7 (GND), U3.10 (GND), U3.6 (CS), U3.7 (MISO), U4.4 (VSS), U4.7 (WP), C1.1, C16.1, C17.1, C2.1, J6.2 (Pin_2)
- net I2C_SDA: now reaches U1.15 (SDA)
- net I2C_SDA: now also IC1.4 (SDA), IC2.4 (SDA), J1.3 (Pin_3), U2.7 (GPIO7), U3.8 (MOSI), U4.5 (SDA), J6.3 (Pin_3), R2.1
- net I2C_SCL: now reaches U1.16 (SCL)
- net I2C_SCL: now also IC1.5 (SCL), IC2.5 (SCL), J1.4 (Pin_4), U2.8 (GPIO8), U3.9 (SCL), U4.6 (SCL), J6.4 (Pin_4), R3.1
- net CJMCU-3935_IRQ_GPIO: now reaches U2.20 (GPIO20)
- net CJMCU-3935_IRQ_GPIO: now also U3.4 (IRQ), J6.5 (Pin_5)
- net SOLAR_IN: now reaches IC2.10 (VIN+)
- net SOLAR_IN: now also R16.1
- net at IC2.8 (VBUS): now also IC2.9 (VIN-), R16.2
- no-connect marks 1 -> 4
Other:
- note added: "address 0x03"
- note added: "address: 0x41"
- note added: "address: 0x44"
- note removed: "EN"
- note removed: "IRQ"
- note removed: "SCL"
- note removed: "SDA"
- moved on the sheet: IC1, IC2, R1, U3, U4

Commit message: hardware schematic draft
Parts:
- removed ANT1: ${DEVICE}, ICs And Semiconductors THD:ANT-BEAD-868, symbol CERN:Sensors/ANT-BEAD-868
- removed R16: R_Small, symbol Device:R_Small
- removed U5: BME280, Package_LGA:Bosch_LGA-8_2.5x2.5mm_P0.65mm_ClockwisePinNumbering, symbol Sensor:BME280
- removed U6: E22-900MM22S, ul_E22-900MM22S:E22-900MM22S_BYT, symbol ul_E22-900MM22S:E22-900MM22S
- added AE1: Antenna, RF_Antenna:Texas_SWRA416_868MHz_915MHz, symbol Device:Antenna
- added C4: 100nF, Capacitor_SMD:C_0603_1608Metric, symbol Device:C_Small
- added IC2: E22-900M22S, E22-900M22S:E22-900M22S, symbol E22-900M22S:E22-900M22S
- added R4, R5: 10k, Resistor_SMD:R_0603_1608Metric, symbol Device:R_Small
- added R6: 0R, Resistor_SMD:R_0603_1608Metric, symbol Device:R_Small
- IC1: value ${DEVICE} -> INA226AIDGST
- IC3: renamed from IC2; value ${DEVICE} -> INA226AIDGST
- J2: renamed from J6; footprint Connector_JST:JST_PH_B4B-PH-K_1x04_P2.00mm_Vertical -> Connector_JST:JST_PH_B5B-PH-K_1x05_P2.00mm_Vertical
- renumbered C16 to C3, C17 to C5, U2 to U1, U1 to U2
Connections:
- net +3V3: now also C4.2, IC2.9 (VCC), R5.2
- net GND: now also C4.1, IC2.1 (GND), IC2.10 (GND), IC2.11 (GND), IC2.12 (GND), IC2.2 (GND), IC2.20 (GND), IC2.22 (GND), IC2.3 (GND), IC2.4 (GND), IC2.5 (GND), R4.2; no longer U3.7 (MISO)
- net SOLAR_IN: now also IC3.8 (VBUS), IC3.9 (VIN-); no longer IC3.10 (VIN+)
- net LORA_NRST: now reaches U1.1 (GPIO1)
- net LORA_NRST: now also IC2.15 (NRST)
- net LORA_NSS: now reaches U1.10 (GPIO10)
- net LORA_NSS: now also IC2.19 (NSS), R5.1
- net SPI_MISO: now reaches U1.2 (GPIO2)
- net SPI_MISO: now also IC2.16 (MISO)
- net LORA_BUSY: now reaches U1.21 (GPIO21)
- net LORA_BUSY: now also IC2.14 (BUSY)
- net SPI_MOSI: now reaches U1.3 (GPIO3)
- net SPI_MOSI: now also IC2.17 (MOSI)
- net SPI_SCK: now reaches U1.4 (GPIO4)
- net SPI_SCK: now also IC2.18 (SCK)
- net LORA_DIO1: now reaches U1.5 (GPIO5)
- net LORA_DIO1: now also IC2.13 (DIO1)
- net BAT_FUSED: now reaches IC1.10 (VIN+)
- net BAT_SYSTEM: now reaches IC1.8 (VBUS)
- net BAT_SYSTEM: now also IC1.9 (VIN-)
- new net: IC2.6 (RXEN), R4.1
- new net: IC2.21 (ANT), R6.2
- new net: IC2.7 (TXEN), IC2.8 (DIO2)
- new net: AE1.1 (A), R6.1
- new net SOLAR+: IC3.10 (VIN+)
- no-connect marks 4 -> 9
Other:
- note added: "INA226AIDGST треба програмно відправляти в deep sleep, щоб він не працював постійно"
- note added: "Модуль BME280"
- note added: "Монітор струму та заряду акумулятора"
- note added: "Програмний sleep"
- note removed: "Контроль заряду акумулятора"
- moved on the sheet: C1, C2, C3, C5, IC1, IC3, J1, J2, R1, R2, R3, U1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

Commit message: hardware improve i2c
Parts:
- removed J1: BME280, Connector_JST:JST_PH_B4B-PH-K_1x04_P2.00mm_Vertical, symbol Connector_Generic:Conn_01x04
- removed J2: CJMCU-3935, Connector_JST:JST_PH_B5B-PH-K_1x05_P2.00mm_Vertical, symbol Connector_Generic:Conn_01x05
- added J1: CJMCU-3935, Connector_JST:JST_PH_B5B-PH-K_1x05_P2.00mm_Vertical, symbol Connector_Generic:Conn_01x05
- added J2: BME280, Connector_JST:JST_PH_B4B-PH-K_1x04_P2.00mm_Vertical, symbol Connector_Generic:Conn_01x04
- added J3: I2C External Modules, Connector_JST:JST_PH_B5B-PH-K_1x05_P2.00mm_Vertical, symbol Connector_Generic:Conn_01x05
- renumbered C4 to C1, C1 to C2, C2 to C4, IC2 to IC1, IC1 to IC2, R4 to R1, R5 to R2, R1 to R3, R6 to R4, R2 to R5, R3 to R6, U3 to U1, U1 to U2, U2 to U3
Connections:
- net +3V3: now also J1.1 (Pin_1), J2.1 (Pin_1), J3.1 (Pin_1)
- net CJMCU-3935_IRQ_GPIO: now also J1.5 (Pin_5); no longer U2.20 (GPIO20)
- net GND: now also J1.2 (Pin_2), J2.2 (Pin_2), J3.2 (Pin_2)
- net I2C_SCL: now also J1.4 (Pin_4), J2.4 (Pin_4), J3.4 (Pin_4)
- net I2C_SDA: now also J1.3 (Pin_3), J2.3 (Pin_3), J3.3 (Pin_3)
- new net WAKE_IRQ: J3.5 (Pin_5), U2.20 (GPIO20)
Other:
- note added: "I2C"
- note added: "SPI"
- note added: "Конектор зовнішніх сенсорів"
- moved on the sheet: AE1, C1, C2, C3, C4, C5, IC1, IC2, IC3, R1, R2, R3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
