File: hardware/untitled.kicad_sch (KiCad schematic)
At the start: 40 parts, among them IC4 TP5000-QFN16, J5 Battary, J7 SMD USB-3.1 Type-C Female 16P, J8 Solar panel, Q1 AO3401A, Q2 MMBT3906, Q3 Q_PMOS_GSD, Q4 Q_PMOS_GSD, Q5 MMBT3904, U9 TPS631000DRLR

Commit message: hardware: power
Parts:
- removed D4, D5: SS14 / SS24, symbol Device:D_Schottky_Small
- removed J7: SMD USB-3.1 Type-C Female 16P, Connector_USB:USB_C_Receptacle_G-Switch_GT-USB-7010ASV, symbol Connector:USB_C_Receptacle_USB2.0_16P
- removed L4: 4.7uH, symbol Device:L
- removed Q1: AO3401A, Package_TO_SOT_SMD:SOT-23, symbol Transistor_FET:AO3401A
- removed Q2: MMBT3906, Package_TO_SOT_SMD:SOT-23, symbol Transistor_BJT:MMBT3906
- removed Q3, Q4: Q_PMOS_GSD, symbol Transistor_FET:Q_PMOS_GSD
- removed Q5: MMBT3904, Package_TO_SOT_SMD:SOT-23, symbol Transistor_BJT:MMBT3904
- removed R11, R12: 5.1kOm, symbol Device:R_Small
- removed R13, R21, R22, R25: 100kOm, symbol Device:R_Small
- removed R23: 47kOm, symbol Device:R_Small
- removed R24: 10kOm, symbol Device:R_Small
- added C1, C5: 100nF, Capacitor_SMD:C_0603_1608Metric, symbol Device:C_Small
- added C2, C3: 1uF, Capacitor_SMD:C_0603_1608Metric, symbol Device:C_Small
- added C8: 4.7uF, Capacitor_SMD:C_0805_2012Metric, symbol Device:C_Small
- added IC3: TPS2121RUXT, TPS2121RUXT:TPS2121RUXT, symbol TPS2121RUXT:TPS2121RUXT
- added J4: USB4105-GF-A-060, USB4105-GF-A-060:GCT_USB4105-GF-A-060, symbol USB4105-GF-A-060:USB4105-GF-A-060
- added L3: IHLP2525CZER4R7M01, footprints:IND_IHLP-2525CZ-01_VIS, symbol ul_IHLP2525CZER4R7M01:IHLP2525CZER4R7M01
- added Q1: IRLML6402TRPBF, Package_TO_SOT_SMD:SOT-23, symbol Transistor_FET:Q_PMOS_GSD
- added R2, R3: 5.1k, Resistor_SMD:R_0603_1608Metric, symbol Device:R_Small
- added R4: 150k, Resistor_SMD:R_0603_1608Metric, symbol Device:R_Small
- added R5: 47k, Resistor_SMD:R_0603_1608Metric, symbol Device:R_Small
- added R6: 80k, Resistor_SMD:R_0603_1608Metric, symbol Device:R_Small
- added U7: LTC4412xS6, Package_TO_SOT_SMD:TSOT-23-6, symbol Power_Management:LTC4412xS6
- C10: renamed from C12; footprint (none) -> Capacitor_SMD:C_0805_2012Metric
- C11: renamed from C14; footprint (none) -> Capacitor_SMD:C_0805_2012Metric
- C12: renamed from C15; footprint (none) -> Capacitor_SMD:C_0805_2012Metric
- C13: renamed from C16; footprint (none) -> Capacitor_SMD:C_0603_1608Metric
- C4: renamed from C9; footprint (none) -> Capacitor_SMD:C_1206_3216Metric
- C6: renamed from C10; footprint (none) -> Capacitor_SMD:C_0603_1608Metric
- C7: renamed from C11; footprint (none) -> Capacitor_SMD:C_1206_3216Metric
- C9: renamed from C13; footprint (none) -> Capacitor_SMD:C_0603_1608Metric
- D1: renamed from D6; footprint (none) -> Diode_SMD:D_SMA
- F1: renamed from F2; value TBD -> MINISMDC300F-2; footprint (none) -> Fuse:Fuse_1812_4532Metric
- R10: renamed from R20; value 91kOm -> 91k; footprint (none) -> Resistor_SMD:R_0603_1608Metric
- R11: renamed from R16; value 10kOm -> 10k; footprint (none) -> Resistor_SMD:R_0603_1608Metric
- R12: renamed from R18; value 4.87kOm -> 4.87k; footprint (none) -> Resistor_SMD:R_0603_1608Metric
- R13: renamed from R19; value 44.2kOm -> 44.2k; footprint (none) -> Resistor_SMD:R_0603_1608Metric
- R7: renamed from R14; value 68mOm -> 68mR; footprint (none) -> Resistor_SMD:R_1206_3216Metric
- R8: renamed from R17; value 511kOm -> 511k; footprint (none) -> Resistor_SMD:R_0603_1608Metric
- R9: renamed from R15; value 10kOm -> 10k; footprint (none) -> Resistor_SMD:R_0603_1608Metric
- renumbered BT2 to BT1, J8 to J3, L3 to L1, U9 to U8
Connections:
- net BAT_FUSED: now also C1.2, Q1.3 (D), U7.1 (VIN)
- net BAT_SYSTEM: now also Q1.2 (S), U7.6 (SENSE)
- net CHARGER_IN: now also C8.2, IC3.1 (OUT_1), IC3.8 (OUT_2)
- net GND: now also C1.1, C2.1, C3.1, C5.1, C8.1, IC3.12 (GND), IC3.3 (CP2), IC3.4 (OV2), IC3.5 (OV1), J4.A1_B12 (GND), J4.B1_A12 (GND), J4.SH1 (SHELL_GND), J4.SH2 (SHELL_GND), J4.SH3 (SHELL_GND), J4.SH4 (SHELL_GND), R2.2, R3.2, R5.1, R6.2, U7.2 (GND)
- net LX_SW: now also L3.1
- net SOLAR_IN: now also C3.2, IC3.2 (IN2)
- net USB_5V: now also C2.2, IC3.7 (IN1), J4.A4_B9 (VBUS), J4.B4_A9 (VBUS), R4.2
- net at C11.1, IC4.8 (VS), R7.2: now also L3.2
- new net: Q1.1 (G), U7.5 (GATE)
- new net: IC3.6 (PR1), R4.1, R5.2
- new net: J4.A5 (CC1), R2.1
- new net: C5.2, IC3.11 (SS)
- new net: J4.B5 (CC2), R3.1
- new net: IC3.10 (ILIM), R6.1
- new net CHARGE_SOURCE_STATUS_OUT: IC3.9 (ST)
- no-connect marks 7 -> 9
Other:
- moved on the sheet: BT1, C10, C11, C12, C13, C4, C6, C7, C9, D1, F1, IC4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

Commit message: hardware root
Parts:
- renumbered C8 to C10, C9 to C11, C10 to C12, C11 to C13, C12 to C14, C13 to C15, C1 to C3, C2 to C4, C3 to C5, C4 to C6, C5 to C7, C6 to C8, C7 to C9, L3 to L2, R8 to R10, R9 to R11, R10 to R12, R11 to R13, R12 to R14, R13 to R15, R2 to R4, R3 to R5, R4 to R6, R5 to R7, R6 to R8, R7 to R9

Commit message: hardware schematic draft
Parts:
- removed C3: 100nF, Capacitor_SMD:C_0603_1608Metric, symbol Device:C_Small
- removed Q1: IRLML6402TRPBF, Package_TO_SOT_SMD:SOT-23, symbol Transistor_FET:Q_PMOS_GSD
- removed U7: LTC4412xS6, Package_TO_SOT_SMD:TSOT-23-6, symbol Power_Management:LTC4412xS6
- added R12: 20mR, Resistor_SMD:R_1206_3216Metric, symbol Device:R_Small
- added R8: 100mR, Resistor_SMD:R_1206_3216Metric, symbol Device:R_Small
- renumbered C8 to C10, C10 to C11, C9 to C12, C11 to C13, C12 to C14, C13 to C15, C14 to C16, C15 to C17, C4 to C6, C5 to C7, C7 to C8, C6 to C9, IC3 to IC4, IC4 to IC5, R6 to R10, R7 to R11, R8 to R13, R9 to R14, R11 to R15, R10 to R16, R13 to R17, R12 to R18, R14 to R19, R15 to R20, R4 to R7, R5 to R9, U8 to U5
Connections:
- net BAT_FUSED: now also R12.2
- net BAT_SYSTEM: now also R12.1
- net SOLAR_IN: now also R8.1; no longer J3.1 (Pin_1)
- new net SOLAR+: J3.1 (Pin_1), R8.2
- no-connect marks 9 -> 7
Other:
- moved on the sheet: C10, C12, C13, C9, F1, J3, J5, L1, R16, R18, U5

Commit message: hardware improve i2c
Parts:
- renumbered C9 to C8, C8 to C9, J3 to J4, J4 to J5, J5 to J6, R16 to R15, R15 to R16
