File: hardware/main_board/main_board.kicad_pcb (KiCad board)
At the start: 2 copper layers, 100 x 62.2 mm, 56 parts, among them IC1 E22-900M22S, IC2 INA226AIDGST, IC3 INA226AIDGST, IC4 TPS2121RUXT, IC5 TP5000-QFN16, J3 I2C External Modules, J4 Solar panel, J5 USB4105-GF-A-060, J6 Battary over BMS, U2 ESP32-C3_SUPERMINI, U3 DS3231SN, U4 FM24CL16B, U5 TPS631000DRLR

Commit message: final schema
Parts:
- removed J6: Battary over BMS, Connector_JST:JST_XH_B3B-XH-A_1x03_P2.50mm_Vertical
- removed U5: TPS631000DRLR, TPS631000DRLR:TPS631000DRLR_TEX
- added C18: 22uF, Capacitor_SMD:C_1206_3216Metric, F.Cu at (95.2, 38.6)
- added C19: 100nF, Capacitor_SMD:C_0603_1608Metric, F.Cu at (70.8, 34.4)
- added C20: 10uF, Capacitor_SMD:C_0805_2012Metric, F.Cu at (87.8, 66.3)
- added C21: 10uF, Capacitor_SMD:C_0805_2012Metric, F.Cu at (87.8, 69.3)
- added C22: 10uF, Capacitor_SMD:C_0805_2012Metric, F.Cu at (87.8, 72.3)
- added C23: 100nF, Capacitor_SMD:C_0603_1608Metric, F.Cu at (70.8, 36.9)
- added J1: EXTERNAL RESET, Connector_JST:JST_EH_B2B-EH-A_1x02_P2.50mm_Vertical, F.Cu at (353.2, 105.8)
- added J2: I2C External Modules, Connector_JST:JST_PH_B5B-PH-K_1x05_P2.00mm_Vertical, F.Cu at (34.8, 87.8)
- added R21: 511k, Resistor_SMD:R_0603_1608Metric, F.Cu at (78.8, 36.9)
- added R22: 10k, Resistor_SMD:R_0603_1608Metric, F.Cu at (78.8, 39.4)
- added R23: 10k, Resistor_SMD:R_0603_1608Metric, F.Cu at (82.8, 19.3)
- added R24: 91k, Resistor_SMD:R_0603_1608Metric, F.Cu at (82.8, 21.8)
- added R25: 4.87k, Resistor_SMD:R_0603_1608Metric, F.Cu at (82.8, 24.3)
- added R26: 44.2k, Resistor_SMD:R_0603_1608Metric, F.Cu at (82.8, 26.8)
- added SW1: RESET, Button_Switch_THT:SW_PUSH_6mm_H5mm, F.Cu at (372.2, 89.2)
- added SW2: BOOT, Button_Switch_THT:SW_PUSH_6mm_H5mm, F.Cu at (372.2, 97.8)
- added U1: ESP32-C3-WROOM-02, RF_Module:ESP32-C3-WROOM-02, F.Cu at (344.2, 95.5)
- C1, C4: value 100nF -> 10uF
- C11: value 4.7uF -> 100nF; footprint Capacitor_SMD:C_0805_2012Metric -> Capacitor_SMD:C_0603_1608Metric
- C12: value 22uF -> 1uF; footprint Capacitor_SMD:C_1206_3216Metric -> Capacitor_SMD:C_0603_1608Metric
- C13, C5: value 100nF -> 1uF
- C14: value 10uF -> 47uF; footprint Capacitor_SMD:C_0805_2012Metric -> Capacitor_SMD:C_1206_3216Metric
- C15, C16: value 10uF -> 100nF; footprint Capacitor_SMD:C_0805_2012Metric -> Capacitor_SMD:C_0603_1608Metric
- C17: value 100nF -> 4.7uF; footprint Capacitor_SMD:C_0603_1608Metric -> Capacitor_SMD:C_0805_2012Metric
- C6, C7: value 1uF -> DNP
- C8: value 47uF -> 100nF; footprint Capacitor_SMD:C_1206_3216Metric -> Capacitor_SMD:C_0603_1608Metric
- D1: value ~ -> SS34; footprint Diode_SMD:D_SMA -> ICs And Semiconductors SMD:DO-214AB
- F1: value MINISMDC300F-2 -> MINISMDC200F-2
- J3: value I2C External Modules -> Solar panel; footprint Connector_JST:JST_PH_B5B-PH-K_1x05_P2.00mm_Vertical -> Connector_JST:JST_XH_B2B-XH-A_1x02_P2.50mm_Vertical
- J4: value Solar panel -> USB4105-GF-A-060; footprint Connector_JST:JST_XH_B2B-XH-A_1x02_P2.50mm_Vertical -> USB4105-GF-A-060:GCT_USB4105-GF-A-060
- J5: value USB4105-GF-A-060 -> Battary over BMS; footprint USB4105-GF-A-060:GCT_USB4105-GF-A-060 -> Connector_JST:JST_XH_B3B-XH-A_1x03_P2.50mm_Vertical
- L2: value IHLP2525CZER4R7M01 -> 4.7 uH; footprint footprints:IND_IHLP-2525CZ-01_VIS -> Inductor_SMD:L_Chilisin_BMRA00050520
- R10: value 150k -> 0R
- R11: value 47k -> 10k
- R12: value 20mR -> 47k; footprint Resistor_SMD:R_1206_3216Metric -> Resistor_SMD:R_0603_1608Metric
- R13: value 80k -> 5.1k
- R14: value 68mR -> 100mR
- R15: value 511k -> 5.1k
- R16: value 10k -> 150k
- R17: value 10k -> 47k
- R18: value 91k -> 20mR; footprint Resistor_SMD:R_0603_1608Metric -> Resistor_SMD:R_1206_3216Metric
- R19: value 4.87k -> 80k
- R20: value 44.2k -> 330mR; footprint Resistor_SMD:R_0603_1608Metric -> Resistor_SMD:R_2512_6332Metric
- R3: value 10k -> 22R
- R4: value 0R -> 22R
- R5: value 4.7k -> 470R
- R6: value 4.7k -> 0R
- R7: value 5.1k -> 4.7k
- R8: value 100mR -> 4.7k; footprint Resistor_SMD:R_1206_3216Metric -> Resistor_SMD:R_0603_1608Metric
- R9: value 5.1k -> 10k
- U2: value ESP32-C3_SUPERMINI -> DS3231SN; footprint esp32c3_super_mini:MODULE_ESP32-C3_SUPERMINI -> Package_SO:SOIC-16W_7.5x10.3mm_P1.27mm
- U3: value DS3231SN -> FM24CL16B; footprint Package_SO:SOIC-16W_7.5x10.3mm_P1.27mm -> Package_SO:SOIC-8_3.9x4.9mm_P1.27mm
- U4: value FM24CL16B -> TPS631000DRLR; footprint Package_SO:SOIC-8_3.9x4.9mm_P1.27mm -> TPS631000DRLR:TPS631000DRLR_TEX
- moved R9 336.6 mm to (363.2, 83.4)
- moved R7 336.2 mm to (363.2, 78.4)
- moved R11 333.6 mm to (367.2, 65.9), turned to 0 degrees
- moved R8 332.3 mm to (363.2, 80.9), turned to 0 degrees
- moved C5 282.7 mm to (355.2, 75.9), turned to 0 degrees
- moved C2 279.9 mm to (355.2, 68.4), turned to 0 degrees
- moved R10 277.7 mm to (315.9, 13.3), turned to 0 degrees
- moved R3 273.2 mm to (363.2, 68.4), turned to 0 degrees
- moved R5 271.8 mm to (363.2, 73.4), turned to 0 degrees
- moved C6 269.3 mm to (307.9, 5.76), turned to 0 degrees
- moved C1 261.4 mm to (355.2, 65.9), turned to 0 degrees
- moved C7 259.9 mm to (307.9, 8.27), turned to 0 degrees
- moved C4 253.2 mm to (307.9, 0.74), turned to 0 degrees
- moved C3 252.2 mm to (307.9, -1.77), turned to 0 degrees
- moved R4 252.1 mm to (363.2, 70.9), turned to 0 degrees
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Connections:
- C1 pad 1: GND -> +3V3
- C1 pad 2: +3V3 -> GND
- C10 pad 1: +3V3 -> GND
- C10 pad 2: GND -> +3V3
- C11 pad 2: /Power/CHARGER_IN -> +3V3
- C12 pad 1: BAT_SYSTEM -> GND
- C12 pad 2: GND -> /Power/USB_5V
- C13 pad 1: BAT_SYSTEM -> GND
- C13 pad 2: GND -> SOLAR_IN
- C14 pad 1: /Power/CHARGER_IN -> +3V3
- C15 pad 1: Net-(IC5-VS) -> GND
- C15 pad 2: GND -> Net-(IC4-SS)
- C16 pad 1: BAT_SYSTEM -> +3V3
- C17 pad 1: Net-(IC5-VREG) -> GND
- C17 pad 2: GND -> /Power/CHARGER_IN
- C2 pad 1: GND -> +3V3
- C2 pad 2: +3V3 -> GND
- C4 pad 1: GND -> +3V3
- C4 pad 2: +3V3 -> GND
- C5 pad 1: GND -> Net-(U1-EN)
- C5 pad 2: +3V3 -> GND
- C6 pad 1: GND -> Net-(C6-Pad1)
- C6 pad 2: /Power/USB_5V -> GND
- C7 pad 1: GND -> Net-(AE1-A)
- C7 pad 2: SOLAR_IN -> GND
- C8 pad 1: +3V3 -> GND
- C8 pad 2: GND -> +3V3
- C9 pad 2: Net-(IC4-SS) -> +3V3
- IC5 pad 14: /Power/STDBY_STATUS -> STDBY_STATUS
- IC5 pad 15: /Power/CHRG_STATUS -> CHRG_STATUS
- J3 pad 1: +3V3 -> SOLAR+
- L1 pad 1: Net-(U5-LX1) -> Net-(U4-LX1)
- L1 pad 2: Net-(U5-LX2) -> Net-(U4-LX2)
- R10 pad 1: Net-(IC4-PR1) -> Net-(C6-Pad1)
- R10 pad 2: /Power/USB_5V -> Net-(AE1-A)
- R11 pad 1: GND -> CHARGE_SOURCE_STATUS_OUT
- R11 pad 2: Net-(IC4-PR1) -> +3V3
- R12 pad 1: BAT_SYSTEM -> /main_board/WAKE_IRQ
- R12 pad 2: BAT_FUSED -> GND
- R13 pad 1: Net-(IC4-ILIM) -> GND
- R13 pad 2: GND -> Net-(J4-CC1)
- R14 pad 1: BAT_SYSTEM -> SOLAR_IN
- R14 pad 2: Net-(IC5-VS) -> SOLAR+
- R15 pad 1: +3V3 -> Net-(J4-CC2)
- R15 pad 2: Net-(U5-FB) -> GND
- R16 pad 1: /Power/CHRG_STATUS -> Net-(IC4-PR1)
- R16 pad 2: +3V3 -> /Power/USB_5V
- R17 pad 1: /Power/STDBY_STATUS -> GND
- R17 pad 2: +3V3 -> Net-(IC4-PR1)
- R18 pad 1: Net-(U5-FB) -> BAT_SYSTEM
- R18 pad 2: GND -> BAT_FUSED
- R19 pad 1: /Power/CHARGER_IN -> Net-(IC4-ILIM)
- R19 pad 2: /Power/NTC_SENSE -> GND
- R20 pad 1: /Power/NTC_SENSE -> BAT_SYSTEM
- R20 pad 2: GND -> Net-(IC5-VS)
- R3 pad 1: CHARGE_SOURCE_STATUS_OUT -> USB_D+
- R3 pad 2: +3V3 -> Net-(U1-IO19)
- R4 pad 1: Net-(AE1-A) -> Net-(U1-IO18)
- R4 pad 2: Net-(IC1-ANT) -> USB_D-
- R5 pad 1: /main_board/I2C_SDA -> Net-(U1-EN)
- R5 pad 2: +3V3 -> Net-(J1-Pin_1)
- R6 pad 1: /main_board/I2C_SCL -> Net-(IC1-ANT)
- R6 pad 2: +3V3 -> Net-(C6-Pad1)
- R7 pad 1: Net-(J5-CC1) -> /main_board/I2C_SDA
- R7 pad 2: GND -> +3V3
- R8 pad 1: SOLAR_IN -> /main_board/I2C_SCL
- R8 pad 2: SOLAR+ -> +3V3
- R9 pad 1: Net-(J5-CC2) -> +3V3
- R9 pad 2: GND -> Net-(U1-EN)
- U2 pad 1: /main_board/WAKE_IRQ -> unconnected-(U2-32KHZ-Pad1)
- U2 pad 10: /main_board/LORA_NSS -> GND
- U2 pad 2: /main_board/SPI_MISO -> +3V3
- U2 pad 3: /main_board/SPI_MOSI -> unconnected-(U2-~{INT}/SQW-Pad3)
- U2 pad 4: /main_board/SPI_SCK -> unconnected-(U2-~{RST}-Pad4)
- U2 pad 5: unconnected-(U2-GPIO5-Pad5) -> GND
- U2 pad 6: CHARGE_SOURCE_STATUS_OUT -> GND
- U2 pad 7: /main_board/I2C_SDA -> GND
- U2 pad 8: /main_board/I2C_SCL -> GND
- U2 pad 9: /main_board/LORA_NRST -> GND
- U3 pad 2: +3V3 -> unconnected-(U3-Pad2)
- U3 pad 4: unconnected-(U3-~{RST}-Pad4) -> GND
- U3 pad 5: GND -> /main_board/I2C_SDA
- U3 pad 6: GND -> /main_board/I2C_SCL
- U3 pad 8: GND -> +3V3
- U4 pad 1: unconnected-(U4-Pad1) -> +3V3
- U4 pad 2: unconnected-(U4-Pad2) -> Net-(U4-LX2)
- U4 pad 3: unconnected-(U4-Pad3) -> Net-(U4-LX1)
- U4 pad 4: GND -> BAT_SYSTEM
- U4 pad 5: /main_board/I2C_SDA -> BAT_SYSTEM
- U4 pad 6: /main_board/I2C_SCL -> GND
- U4 pad 8: +3V3 -> Net-(U4-FB)
Routing:
- net BAT_SYSTEM: track 41.5 -> 0.00 mm
- net /Power/USB_5V: track 22.8 -> 0.00 mm
- net +3V3: track 19.2 -> 0.00 mm
- net SOLAR_IN: track 16.6 -> 0.00 mm
- net GND: track 9.06 -> 0.00 mm
- net Net-(IC5-VS): track 9.05 -> 0.00 mm
- net Net-(IC4-PR1): track 7.99 -> 0.00 mm
- net /Power/CHARGER_IN: track 5.77 -> 0.00 mm
- net /Power/BAT_RAW: track 5.50 -> 0.00 mm
- net /Power/LX_SW: track 4.95 -> 0.00 mm
- net SOLAR+: track 4.89 -> 0.00 mm
- net Net-(U5-FB): track 4.83 -> 0.00 mm
- net BAT_FUSED: track 4.02 -> 0.00 mm
- net Net-(U5-LX2): track 2.96 -> 0.00 mm
- net Net-(U5-LX1): track 2.75 -> 0.00 mm
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- removed copper zone on B.Cu, net GND
- removed copper zone on F.Cu, net GND
Other:
- board outline removed

Commit message: hw start board
Parts:
- removed J4: USB4105-GF-A-060, USB4105-GF-A-060:GCT_USB4105-GF-A-060
- added J6: USB4105-GF-A-060, Connector_USB:USB_C_Receptacle_GCT_USB4105-xx-A_16P_TopMnt_Horizontal, F.Cu at (106.5, 101.2)
- added R27: 44.2k, Resistor_SMD:R_0603_1608Metric, F.Cu at (156.8, 112.9)
- C5: value 1uF -> DNP
- C6: value DNP -> 1uF
- R1, R11: value 10k -> 0R
- R10: value 0R -> 10k
- R12: value 47k -> 10k
- R13: value 5.1k -> 47k
- R14: value 100mR -> 5.1k; footprint Resistor_SMD:R_1206_3216Metric -> Resistor_SMD:R_0603_1608Metric
- R15: value 5.1k -> 100mR; footprint Resistor_SMD:R_0603_1608Metric -> Resistor_SMD:R_1206_3216Metric
- R16: value 150k -> 5.1k
- R17: value 47k -> 150k
- R18: value 20mR -> 47k; footprint Resistor_SMD:R_1206_3216Metric -> Resistor_SMD:R_0603_1608Metric
- R19: value 80k -> 20mR; footprint Resistor_SMD:R_0603_1608Metric -> Resistor_SMD:R_1206_3216Metric
- R20: value 330mR -> 80k; footprint Resistor_SMD:R_2512_6332Metric -> Resistor_SMD:R_0603_1608Metric
- R21: value 511k -> 330mR; footprint Resistor_SMD:R_0603_1608Metric -> Resistor_SMD:R_2512_6332Metric
- R22: value 10k -> 511k
- R24: value 91k -> 10k
- R25: value 4.87k -> 91k
- R26: value 44.2k -> 4.87k
- R3: value 22R -> 10k
- R5: value 470R -> 22R
- R6: value 0R -> 470R
- R7: value 4.7k -> 0R
- R9: value 10k -> 4.7k
- moved SW1 270.4 mm to (102.7, 67.1)
- moved SW2 259.5 mm to (113.4, 78.9)
- moved R9 249.4 mm to (114.0, 71.8), turned to 90 degrees
- moved R8 246.6 mm to (116.8, 70.2), turned to 90 degrees
- moved J1 245.8 mm to (108.5, 82.5), turned to -90 degrees
- moved C1 239.1 mm to (116.1, 65.7), turned to 180 degrees
- moved C2 237.9 mm to (117.3, 63.6), turned to 180 degrees
- moved R5 223.3 mm to (139.9, 71.3)
- moved R4 223.2 mm to (140.0, 69.5), turned to 180 degrees
- moved R6 220.2 mm to (109.0, 78.5), turned to 180 degrees
- moved U1 217.1 mm to (128.7, 69.6)
- moved R10 215.8 mm to (108.9, 74.4)
- moved C6 211.1 mm to (109.0, 76.5), turned to 180 degrees
- moved R11 187.6 mm to (179.6, 66.2), turned to 90 degrees
- moved R1 181.9 mm to (140.0, 72.8), turned to 180 degrees
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Connections:
- net Net-(IC1-DIO2) renamed /main_board/LORA_TXEN
- C5 pad 1: Net-(U1-EN) -> Net-(C5-Pad1)
- C6 pad 1: Net-(C6-Pad1) -> Net-(U1-EN)
- IC1 pad 6: Net-(IC1-RXEN) -> /main_board/LORA_RXEN
- R1 pad 1: Net-(IC1-RXEN) -> /main_board/LORA_RXEN
- R1 pad 2: GND -> Net-(U1-IO21/TXD)
- R10 pad 1: Net-(C6-Pad1) -> +3V3
- R10 pad 2: Net-(AE1-A) -> Net-(U1-EN)
- R11 pad 1: CHARGE_SOURCE_STATUS_OUT -> Net-(C5-Pad1)
- R11 pad 2: +3V3 -> Net-(AE1-A)
- R12 pad 1: /main_board/WAKE_IRQ -> CHARGE_SOURCE_STATUS_OUT
- R12 pad 2: GND -> +3V3
- R13 pad 1: GND -> /main_board/WAKE_IRQ
- R13 pad 2: Net-(J4-CC1) -> GND
- R14 pad 1: SOLAR_IN -> GND
- R14 pad 2: SOLAR+ -> Net-(J6-CC1)
- R15 pad 1: Net-(J4-CC2) -> SOLAR_IN
- R15 pad 2: GND -> SOLAR+
- R16 pad 1: Net-(IC4-PR1) -> Net-(J6-CC2)
- R16 pad 2: /Power/USB_5V -> GND
- R17 pad 1: GND -> Net-(IC4-PR1)
- R17 pad 2: Net-(IC4-PR1) -> /Power/USB_5V
- R18 pad 1: BAT_SYSTEM -> GND
- R18 pad 2: BAT_FUSED -> Net-(IC4-PR1)
- R19 pad 1: Net-(IC4-ILIM) -> BAT_SYSTEM
- R19 pad 2: GND -> BAT_FUSED
- R2 pad 1: /main_board/LORA_NSS -> /main_board/LORA_RXEN
- R2 pad 2: +3V3 -> GND
- R20 pad 1: BAT_SYSTEM -> Net-(IC4-ILIM)
- R20 pad 2: Net-(IC5-VS) -> GND
- R21 pad 1: +3V3 -> BAT_SYSTEM
- R21 pad 2: Net-(U4-FB) -> Net-(IC5-VS)
- R22 pad 1: CHRG_STATUS -> +3V3
- R22 pad 2: +3V3 -> Net-(U4-FB)
- R23 pad 1: STDBY_STATUS -> CHRG_STATUS
- R24 pad 1: Net-(U4-FB) -> STDBY_STATUS
- R24 pad 2: GND -> +3V3
- R25 pad 1: /Power/CHARGER_IN -> Net-(U4-FB)
- R25 pad 2: /Power/NTC_SENSE -> GND
- R26 pad 1: /Power/NTC_SENSE -> /Power/CHARGER_IN
- R26 pad 2: GND -> /Power/NTC_SENSE
- R3 pad 1: USB_D+ -> /main_board/LORA_NSS
- R3 pad 2: Net-(U1-IO19) -> +3V3
- R4 pad 1: Net-(U1-IO18) -> USB_D+
- R4 pad 2: USB_D- -> Net-(U1-IO19)
- R5 pad 1: Net-(U1-EN) -> Net-(U1-IO18)
- R5 pad 2: Net-(J1-Pin_1) -> USB_D-
- R6 pad 1: Net-(IC1-ANT) -> Net-(U1-EN)
- R6 pad 2: Net-(C6-Pad1) -> Net-(J1-Pin_1)
- R7 pad 1: /main_board/I2C_SDA -> Net-(IC1-ANT)
- R7 pad 2: +3V3 -> Net-(C5-Pad1)
- R8 pad 1: /main_board/I2C_SCL -> /main_board/I2C_SDA
- R9 pad 1: +3V3 -> /main_board/I2C_SCL
- R9 pad 2: Net-(U1-EN) -> +3V3
- U1 pad 12: unconnected-(U1-IO21/TXD-Pad12) -> Net-(U1-IO21/TXD)
Routing:
- net /Power/USB_5V: track 0.00 -> 47.4 mm
- net +3V3: track 0.00 -> 38.3 mm
- net Net-(U1-EN): track 0.00 -> 34.7 mm, vias 0 -> 1
- net /main_board/WAKE_IRQ: track 0.00 -> 32.6 mm, vias 0 -> 2
- net BAT_SYSTEM: track 0.00 -> 31.2 mm
- net /Power/CHARGER_IN: track 0.00 -> 26.2 mm
- net Net-(IC5-VS): track 0.00 -> 17.9 mm
- net /main_board/LORA_NRST: track 0.00 -> 15.0 mm
- net USB_D+: track 0.00 -> 14.9 mm, vias 0 -> 2
- net USB_D-: track 0.00 -> 13.5 mm, vias 0 -> 2
- net /Power/LX_SW: track 0.00 -> 10.4 mm
- net Net-(C5-Pad1): track 0.00 -> 9.30 mm
- net GND: track 0.00 -> 7.43 mm
- net /Power/BAT_RAW: track 0.00 -> 6.63 mm
- net /main_board/I2C_SCL: track 0.00 -> 5.88 mm
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- added copper zone on B.Cu, net GND
- added copper zone on F.Cu, net GND
Other:
- board outline added: 99.4 x 85 mm

Commit message: hw pcb
Parts:
- added TP1: TP_SOLAR_IN, TestPoint:TestPoint_Pad_D1.0mm, F.Cu at (49.8, 49.1)
- added TP10: TP_GND_RF, TestPoint:TestPoint_Pad_D1.0mm, F.Cu at (213.6, 70.4)
- added TP2: TP_BAT_RAW, TestPoint:TestPoint_Pad_D1.0mm, F.Cu at (33.5, 92.0)
- added TP3: TP_BAT_FUSED, TestPoint:TestPoint_Pad_D1.0mm, F.Cu at (40.6, 97.0)
- added TP4: TP_BAT_SYSTEM, TestPoint:TestPoint_Pad_D1.0mm, F.Cu at (46.5, 93.2)
- added TP5: TP_USB_5V, TestPoint:TestPoint_Pad_D1.0mm, F.Cu at (31.9, 48.5)
- added TP6: TP_CHARGER_IN, TestPoint:TestPoint_Pad_D1.0mm, F.Cu at (143.0, 26.7)
- added TP7: TP_BAT_SYSTEM, TestPoint:TestPoint_Pad_D1.0mm, F.Cu at (63.3, 95.9)
- added TP8: TP_3V3, TestPoint:TestPoint_Pad_D1.0mm, F.Cu at (53.5, 83.6)
- added TP9: TP_GND_PWR, TestPoint:TestPoint_Pad_D1.0mm, F.Cu at (204.7, 120.4)
- BT1: moved to B.Cu
- J3: footprint Connector_JST:JST_XH_B2B-XH-A_1x02_P2.50mm_Vertical -> TerminalBlock_Philmore:TerminalBlock_Philmore_TB132_1x02_P5.00mm_Horizontal
- moved R1 180.1 mm to (-39.9, 62.5), turned to 90 degrees
- moved R12 172.8 mm to (-47.4, 54.5), turned to 90 degrees
- moved C1 163.5 mm to (-47.4, 70.5), turned to 90 degrees
- moved C2 162.4 mm to (-44.9, 70.5), turned to 90 degrees
- moved R8 157.1 mm to (-39.9, 58.5)
- moved R6 155.1 mm to (-44.9, 58.5), turned to 90 degrees
- moved SW2 154.9 mm to (-38.1, 46.4), turned to 90 degrees
- moved R9 152.0 mm to (-37.3, 58.5)
- moved SW1 150.7 mm to (-46.6, 46.4), turned to 90 degrees
- moved R10 144.6 mm to (-34.8, 58.5), turned to 90 degrees
- moved C6 143.9 mm to (-34.8, 70.5), turned to 90 degrees
- moved J1 141.3 mm to (-30.0, 54.3), turned to 90 degrees
- moved R4 107.1 mm to (34.0, 53.7), turned to -90 degrees
- moved R5 105.8 mm to (35.8, 52.3), turned to 90 degrees
- moved C22 99.0 mm to (60.8, 94.3), turned to 180 degrees
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Routing:
- net BT_CR2032: track 0.00 -> 38.5 mm, vias 0 -> 1
- net Net-(U1-EN): track 34.7 -> 0.00 mm, vias 1 -> 0
- net /main_board/WAKE_IRQ: track 32.6 -> 0.00 mm, vias 2 -> 0
- net /Power/CHARGER_IN: track 26.2 -> 7.52 mm
- net SOLAR_IN: track 2.33 -> 19.4 mm
- net /main_board/LORA_NRST: track 15.0 -> 0.00 mm
- net Net-(U1-IO18): track 1.73 -> 13.7 mm, vias 0 -> 2
- net Net-(U1-IO19): track 1.75 -> 12.5 mm, vias 0 -> 2
- net Net-(IC5-VS): track 17.9 -> 7.76 mm
- net Net-(C5-Pad1): track 9.30 -> 0.00 mm
- net /Power/USB_5V: track 47.4 -> 56.1 mm
- net USB_D+: track 14.9 -> 7.96 mm, vias 2 -> 0
- net /main_board/I2C_SCL: track 5.88 -> 0.00 mm
- net GND: track 7.43 -> 13.1 mm, vias 0 -> 5
- net Net-(AE1-A): track 4.56 -> 0.00 mm
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- added copper zone on F.Cu, net +3V3
- added copper zone on F.Cu, net /Power/LX_SW
- added copper zone on F.Cu, net BAT_SYSTEM
- added copper zone on F.Cu, net Net-(IC5-VS)
Other:
- board outline removed

Commit message: hw pcb v0.2
Parts:
- removed C10: 100nF, Capacitor_SMD:C_0603_1608Metric
- removed J1: EXTERNAL RESET, Connector_JST:JST_EH_B2B-EH-A_1x02_P2.50mm_Vertical
- removed R6: 470R, Resistor_SMD:R_0603_1608Metric
- removed SW1: RESET, Button_Switch_THT:SW_PUSH_6mm_H5mm
- removed SW2: BOOT, Button_Switch_THT:SW_PUSH_6mm_H5mm
- removed the TP10 at (213.6, 70.4)
- removed U3: FM24CL16B, Package_SO:SOIC-8_3.9x4.9mm_P1.27mm
- added TP10: GND, TestPoint:TestPoint_Pad_D1.5mm, F.Cu at (96.0, 94.6)
- added TP10: BOOT, TestPoint:TestPoint_Pad_D1.5mm, F.Cu at (99.6, 87.9)
- TP6: value TP_CHARGER_IN -> EN; footprint TestPoint:TestPoint_Pad_D1.0mm -> TestPoint:TestPoint_Pad_D1.5mm
- moved R8 152.2 mm to (110.8, 79.9), turned to 0 degrees
- moved R9 150.2 mm to (110.8, 82.8), turned to 0 degrees
- moved R12 145.8 mm to (94.5, 88.2), turned to -90 degrees
- moved TP9 145.7 mm to (80.9, 43.6)
- moved R1 138.9 mm to (99.1, 64.8), turned to 180 degrees
- moved C1 136.9 mm to (88.4, 88.2), turned to -90 degrees
- moved C2 135.9 mm to (89.9, 88.1), turned to -90 degrees
- moved C4 131.6 mm to (129.8, 42.4), turned to 180 degrees
- moved C3 129.7 mm to (129.8, 40.9), turned to 0 degrees
- moved R10 129.7 mm to (91.4, 88.1)
- moved C6 129.0 mm to (93.0, 88.2), turned to -90 degrees
- moved R2 126.1 mm to (135.5, 42.6), turned to 0 degrees
- moved R3 121.4 mm to (139.3, 59.5), turned to 0 degrees
- moved R26 120.1 mm to (118.8, 106.6), turned to 90 degrees
- moved C7 119.3 mm to (146.6, 53.9), turned to 180 degrees
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Connections:
- TP6 pad 1: /Power/CHARGER_IN -> Net-(U1-EN)
Routing:
- net /Power/NTC_SENSE: track 0.00 -> 45.3 mm
- net BAT_FUSED: track 5.91 -> 33.3 mm, vias 0 -> 2
- net /main_board/I2C_SDA: track 0.00 -> 16.8 mm
- net /Power/CHARGER_IN: track 7.52 -> 22.0 mm
- net /main_board/I2C_SCL: track 0.00 -> 14.1 mm
- net BAT_SYSTEM: track 32.6 -> 44.1 mm
- net GND: track 13.1 -> 23.9 mm, vias 5 -> 9
- net Net-(U1-EN): track 0.00 -> 8.01 mm
- net +3V3: track 40.0 -> 47.8 mm
- net Net-(C5-Pad1): track 0.00 -> 5.32 mm
- net Net-(AE1-A): track 0.00 -> 3.73 mm
- net Net-(U1-IO21/TXD): track 0.00 -> 3.70 mm
- net /main_board/WAKE_IRQ: track 0.00 -> 3.26 mm
- net /main_board/LORA_NRST: track 0.00 -> 2.95 mm
- net CHARGE_SOURCE_STATUS_OUT: track 0.00 -> 1.92 mm
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Other:
- board outline added: 95.3 x 70.9 mm
- board text added: "3v3"

Commit message: hw pcb v0.3
Parts:
- moved R13 43.8 mm to (150.0, 79.3), turned to 0 degrees
- moved J2 30.5 mm to (141.2, 82.5), turned to 0 degrees
- moved AE1 20.5 mm to (161.8, 67.6), turned to -90 degrees
- moved R7 8.98 mm to (153.9, 64.3), turned to 90 degrees
- moved C7 8.91 mm to (155.3, 56.1), turned to 90 degrees
- moved R11 5.69 mm to (153.9, 59.4), turned to 90 degrees
- moved TP6 4.78 mm to (99.6, 91.6)
- moved C5 4.11 mm to (151.2, 61.9), turned to 180 degrees
Routing:
- net +3V3: track 47.8 -> 280.8 mm, vias 0 -> 6
- net /main_board/I2C_SCL: track 14.1 -> 173.6 mm, vias 0 -> 5
- net /main_board/WAKE_IRQ: track 3.26 -> 154.2 mm, vias 0 -> 2
- net /main_board/I2C_SDA: track 16.8 -> 167.1 mm, vias 0 -> 3
- net /Power/CHARGER_IN: track 22.0 -> 165.7 mm, vias 0 -> 4
- net CHARGE_SOURCE_STATUS_OUT: track 1.92 -> 123.8 mm, vias 0 -> 2
- net /main_board/LORA_RXEN: track 1.92 -> 48.2 mm
- net Net-(IC1-ANT): track 1.78 -> 14.0 mm
- net Net-(U1-EN): track 8.01 -> 12.5 mm
- net BT_CR2032: track 38.5 -> 42.1 mm
- net GND: vias 9 -> 11
Other:
- board size 95.3 x 70.9 mm -> 95.3 x 71.6 mm

Commit message: hw v0.4
Parts:
- moved IC3 0.80 mm to (109.7, 45.3)
- moved C17 0.07 mm to (117.9, 48.7)
- renumbered TP10 to TP11
Routing:
- net /main_board/SPI_SCK: track 0.00 -> 85.5 mm, vias 0 -> 2
- net /main_board/LORA_NRST: track 2.95 -> 87.8 mm, vias 0 -> 2
- net /main_board/SPI_MOSI: track 0.00 -> 84.3 mm, vias 0 -> 4
- net /main_board/SPI_MISO: track 0.00 -> 66.0 mm, vias 0 -> 2
- net /main_board/LORA_BUSY: track 0.00 -> 55.6 mm, vias 0 -> 2
- net /main_board/LORA_NSS: track 1.75 -> 51.2 mm, vias 0 -> 2
- net /main_board/LORA_DIO1: track 0.00 -> 42.3 mm
- net GND: track 23.9 -> 40.4 mm, vias 11 -> 34
- net /main_board/LORA_TXEN: track 0.00 -> 1.27 mm
- net /main_board/I2C_SCL: track 173.6 -> 172.9 mm
- net SOLAR+: track 8.16 -> 8.69 mm

Commit message: hw v0.5
Parts:
- J6: footprint Connector_USB:USB_C_Receptacle_GCT_USB4105-xx-A_16P_TopMnt_Horizontal -> Connector_USB:USB_C_Receptacle_HRO_TYPE-C-31-M-12
- TP10: value BOOT -> ESP32_BOOT
- TP6: value EN -> ESP32_EN
Routing:
- net GND: track 40.4 -> 42.4 mm
- net /Power/USB_5V: track 56.1 -> 55.5 mm

Commit message: hw v0.6
Parts:
- moved TP1 4.69 mm to (109.1, 49.8)
- moved TP6 0.57 mm to (99.3, 91.1)
Routing:
- net SOLAR_IN: track 19.6 -> 16.9 mm
- net GND: vias 34 -> 33
Changed lines of the file:
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@@
 		(tags "capacitor")
 		(property "Reference" "C6"
-			(at 2.527 -0.127 90)
+			(at 2.781 -0.127 90)
 			(layer "F.SilkS")
 			(effects
@@
 		)
 		(fp_text user "${REFERENCE}"
-			(at 0 -1.65 0)
-			(layer "F.Fab")
+			(at -3.175 -0.508 0)
+			(layer "F.SilkS")
 			(effects
 				(font
@@
 		(fp_text user "${REFERENCE}"
 			(at 3.048 -0.508 0)
-			(layer "F.Fab")
+			(layer "F.SilkS")
 			(effects
 				(font
@@
 		)
 		(fp_text user "eByte"
-			(at -1.27 0 90)
+			(at 0.269 2.033 180)
 			(layer "F.SilkS")
 			(effects
@@
 		)
 		(fp_text user "E22-900M22S"
-			(at 2.54 3.81 90)
+			(at 2.936 2.668 180)
 			(layer "F.SilkS")
 			(effects
@@
 	(footprint "TestPoint:TestPoint_Pad_D1.5mm"
 		(layer "F.Cu")
-		(at 99.568 91.567)
+		(at 99.314 91.059)
 		(descr "SMD pad as test Point, diameter 1.5mm")
 		(tags "test point SMD pad")
@@
 		)
 		(fp_text user "${REFERENCE}"
-			(at 0 -1.65 0)
-			(layer "F.Fab")
+			(at 0 2.032 0)
+			(layer "F.SilkS")
 			(effects
 				(font
@@
 		(tags "test point SMD pad")
 		(property "Reference" "TP2"
-			(at 0 -1.448 0)
+			(at 0.3196 -1.5774 0)
 			(layer "F.SilkS")
 			(effects
@@
 	(footprint "TestPoint:TestPoint_Pad_D1.0mm"
 		(layer "F.Cu")
-		(at 105.0904 52.2319)
+		(at 109.093 49.784)
 		(descr "SMD pad as test Point, diameter 1.0mm")
 		(tags "test point SMD pad")
 		(property "Reference" "TP1"
-			(at 0 -1.448 0)
+			(at -1.778 -0.254 90)
 			(layer "F.SilkS")
 			(effects
@@
 			(effects
 				(font
-					(size 0.787402 0.787402)
+					(size 1 1)
 					(thickness 0.15)
 				)
@@
 		(tags "test point SMD pad")
 		(property "Reference" "TP3"
-			(at 0 -1.448 0)
+			(at -0.0656 -1.6776 0)
 			(layer "F.SilkS")
 			(effects
@@
 	)
 	(via
-		(at 95.758 89.027)
-		(size 0.6)
-		(drill 0.3)
-		(layers "F.Cu" "B.Cu")
-		(free yes)
-		(net "GND")
-	)
-	(via
 		(at 109.4665 45.7275)
 		(size 0.6)
@@
 	)
 	(segment
-		(start 113.5594 49.6679)
-		(end 108.1624 49.6679)
-		(width 0.5)
-		(layer "F.Cu")
-		(net "SOLAR_IN")
-	)
-	(segment
-		(start 105.0904 51.2159)
-		(end 105.0904 52.2319)
-		(width 1)
+		(start 107.553 45.864)
+		(end 107.528 45.839)
+		(width 0.25)
 		(layer "F.Cu")
 		(net "SOLAR_IN")
 	)
 	(segment
-		(start 108.6624 45.9234)
-		(end 108.078 45.339)
+		(start 108.6624 45.559796)
+		(end 108.441604 45.339)
 		(width 0.25)
 		(layer "F.Cu")
@@
 	(segment
 		(start 105.0904 49.8229)
-		(end 105.0904 51.2159)
-		(width 1)
+		(end 106.5754 49.8229)
+		(width 0.5)
 		(layer "F.Cu")
 		(net "SOLAR_IN")
 	)
 	(segment
-		(start 105.0904 49.8229)
-		(end 106.5754 49.8229)
-		(width 0.5)
+		(start 108.6624 46.7859)
+		(end 108.6624 45.559796)
+		(width 0.25)
 		(layer "F.Cu")
 		(net "SOLAR_IN")
@@
 	)
 	(segment
-		(start 108.078 45.339)
+		(start 108.441604 45.339)
 		(end 107.528 45.339)
 		(width 0.25)
@@
 	)
 	(segment
-		(start 106.6144 51.2159)
-		(end 105.0904 51.2159)
-		(width 0.5)
-		(layer "F.Cu")
-		(net "SOLAR_IN")
-	)
-	(segment
 		(start 106.5754 49.8229)
 		(end 108.6624 47.7359)
@@
 	)
 	(segment
-		(start 108.6624 46.7859)
-		(end 108.6624 45.9234)
-		(width 0.25)
+		(start 112.9344 49.8229)
+		(end 113.0894 49.6679)
+		(width 0.5)
 		(layer "F.Cu")
 		(net "SOLAR_IN")
 	)
 	(segment
-		(start 108.1624 49.6679)
-		(end 106.6144 51.2159)
+		(start 105.0904 49.8229)
+		(end 112.9344 49.8229)
 		(width 0.5)
 		(layer "F.Cu")
@@
 		(layer "F.Cu")
 		(net "SOLAR_IN")
+	)
+	(segment
+		(start 113.0894 49.6679)
+		(end 113.5594 49.6679)
+		(width 0.5)
+		(layer "F.Cu")
+		(net "SOLAR_IN")
