File: hardware/main_board/untitled.kicad_sch (KiCad schematic)
At the start: 37 parts, among them IC4 TPS2121RUXT, IC5 TP5000-QFN16, J4 Solar panel, J5 USB4105-GF-A-060, J6 Battary over BMS, U5 TPS631000DRLR

Commit message: final schema
Parts:
- removed L2: IHLP2525CZER4R7M01, footprints:IND_IHLP-2525CZ-01_VIS, symbol ul_IHLP2525CZER4R7M01:IHLP2525CZER4R7M01
- removed R7: 5.1k, Resistor_SMD:R_0603_1608Metric, symbol Device:R_Small
- added L2: 4.7 uH, Inductor_SMD:L_Chilisin_BMRA00050520, symbol Device:L_Small
- added R14: 5.1k, Resistor_SMD:R_0603_1608Metric, symbol Device:R_Small
- C12: renamed from C6; Comment (none) -> X7R, ±10%, 16 V
- C13: renamed from C7; Comment (none) -> X7R, ±10%, 16 V
- C14: renamed from C8; Comment (none) -> X5R/X7R, ≥6.3 V, preferably 10 V; check DC-bias derating
- C15: renamed from C9; Comment (none) -> X7R, ±10%, 16 V
- C16: renamed from C10; Comment (none) -> X7R, ±10%, 16 V
- C17: renamed from C11; Comment (none) -> X7R/X5R, ≥10 V, 16 V preferred
- C18: renamed from C12; Comment (none) -> X5R/X7R, ≥6.3 V, preferably 10 V
- C19: renamed from C13; Comment (none) -> X7R, ±10%, 16 V
- C20: renamed from C14; Comment (none) -> X5R/X7R, ≥10 V, 16 V preferred
- C21: renamed from C15; Comment (none) -> X5R/X7R, ≥6.3 V, preferably 10 V
- C22: renamed from C16; Comment (none) -> X5R/X7R, ≥6.3 V, preferably 10 V
- C23: renamed from C17; Comment (none) -> X7R, ±10%, 16 V
- D1: value (none) -> SS34; footprint Diode_SMD:D_SMA -> ICs And Semiconductors SMD:DO-214AB
- F1: value MINISMDC300F-2 -> MINISMDC200F-2
- R15: renamed from R8; Comment (none) -> current sense, ±1% або краще, low-TCR ≤50 ppm/°C, ≥0.5 W
- R17: renamed from R10; Comment (none) -> Priority / threshold divider, ±1%
- R18: renamed from R11; Comment (none) -> Priority / threshold divider, ±1%
- R19: renamed from R12; Comment (none) -> current sense, ±1%/±0.5%, low-TCR ≤50 ppm/°C, ≥0.5 W recomm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
- R20: renamed from R13; Comment (none) -> TPS2121 ILIM programming resistor, ±1%. Value change affect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
- R21: renamed from R14; value 68mR -> 330mR; footprint Resistor_SMD:R_1206_3216Metric -> Resistor_SMD:R_2512_6332Metric; Comment (none) -> current/charge setting resistor, ±1%, low-TCR, ≥1 W; Why (none) -> Обмежуємо струм до максимально допустимого від сонячної пан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
- R22: renamed from R15; Comment (none) -> VOUT feedback divider — precision resistors, ±0.5% or bette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
- R25: renamed from R18; Comment (none) -> VOUT feedback divider — precision resistors, ±0.5% or bette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
- R26: renamed from R19; Comment (none) -> Programming / sensing network — ±1%, do not substitute with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
- R27: renamed from R20; Comment (none) -> Programming / sensing network — ±1%, do not substitute with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
- renumbered J4 to J3, J5 to J4, J6 to J5, R9 to R16, R16 to R23, R17 to R24, U5 to U4
Connections:
- net GND: now also R14.1
- net LX_SW: now also L2.1
- net at C21.1, IC5.8 (VS), R21.2: now also L2.2
- net at J4.A5 (CC1): now also R14.2
- net USB_D+: now reaches J4.A6 (DP1)
- net USB_D+: now also J4.B6 (DP2)
- net USB_D-: now reaches J4.A7 (DN1)
- net USB_D-: now also J4.B7 (DN2)
- no-connect marks 7 -> 3
Other:
- note added: "1S LiFePO4 charger. Battery chemistry: LiFePO4, nominal 3.2 V."
- note added: "Power source priority: USB_5V has priority over SOLAR_IN. When USB power is present, Solar input must not supply the system."
- note added: "Resistors unless otherwise specified: ±1%, ≥0.1 W, ≤100 ppm/°C. 100 nF / 1 µF MLCC: X7R, ±10%, voltage rating as specified. Bulk MLCC ≥4.7 µF: X5R or X7R, ±20%, verify effective capacitance under DC bias. Do not use Y5V/Z5U capacitors. DNP = Do Not Populate. All components intended for outdoor operation: industrial temperature grade preferred (-40…+85 °C or better)."
- title: (none) -> Power
- moved on the sheet: C21, C22, R16, R21

Commit message: hw start board
Parts:
- removed J4: USB4105-GF-A-060, USB4105-GF-A-060:GCT_USB4105-GF-A-060, symbol USB4105-GF-A-060:USB4105-GF-A-060
- added J6: USB4105-GF-A-060, Connector_USB:USB_C_Receptacle_GCT_USB4105-xx-A_16P_TopMnt_Horizontal, symbol Connector:USB_C_Receptacle_USB2.0_16P
Connections:
- net GND: now also J6.A1 (GND), J6.A12 (GND), J6.B1 (GND), J6.B12 (GND), J6.SH (SHIELD)
- net USB_5V: now also J6.A4 (VBUS), J6.A9 (VBUS), J6.B4 (VBUS), J6.B9 (VBUS)
- net USB_D+: now also J6.A6 (D+), J6.B6 (D+)
- net USB_D-: now also J6.A7 (D-), J6.B7 (D-)
- net at R14.2: now also J6.A5 (CC1)
- net at R16.1: now also J6.B5 (CC2)
Other:
- moved on the sheet: J3, R15

Commit message: hw pcb
Parts:
- added TP1: TP_SOLAR_IN, TestPoint:TestPoint_Pad_D1.0mm, symbol Connector:TestPoint_Small
- added TP2: TP_BAT_RAW, TestPoint:TestPoint_Pad_D1.0mm, symbol Connector:TestPoint_Small
- added TP3: TP_BAT_FUSED, TestPoint:TestPoint_Pad_D1.0mm, symbol Connector:TestPoint_Small
- added TP4, TP7: TP_BAT_SYSTEM, TestPoint:TestPoint_Pad_D1.0mm, symbol Connector:TestPoint_Small
- added TP5: TP_USB_5V, TestPoint:TestPoint_Pad_D1.0mm, symbol Connector:TestPoint_Small
- added TP6: TP_CHARGER_IN, TestPoint:TestPoint_Pad_D1.0mm, symbol Connector:TestPoint_Small
- added TP8: TP_3V3, TestPoint:TestPoint_Pad_D1.0mm, symbol Connector:TestPoint_Small
- added TP9: TP_GND_PWR, TestPoint:TestPoint_Pad_D1.0mm, symbol Connector:TestPoint_Small
- J3: footprint Connector_JST:JST_XH_B2B-XH-A_1x02_P2.50mm_Vertical -> TerminalBlock_Philmore:TerminalBlock_Philmore_TB132_1x02_P5.00mm_Horizontal
Connections:
- net +3V3: now also TP8.1
- net BAT_FUSED: now also TP3.1
- net BAT_RAW: now also TP2.1
- net BAT_SYSTEM: now also TP4.1, TP7.1
- net CHARGER_IN: now also TP6.1
- net GND: now also TP9.1
- net SOLAR_IN: now also TP1.1
- net USB_5V: now also TP5.1

Commit message: hw pcb v0.2
Parts:
- removed TP6: TP_CHARGER_IN, TestPoint:TestPoint_Pad_D1.0mm, symbol Connector:TestPoint_Small
Changed lines of the file:
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@@
 	)
 	(junction
-		(at 163.83 66.04)
-		(diameter 0)
-		(color 0 0 0 0)
-	)
-	(junction
 		(at 50.8 27.94)
 		(diameter 0)
@@
 	(wire
 		(pts
-			(xy 163.83 64.77) (xy 163.83 66.04)
-		)
-		(stroke
-			(width 0)
-			(type default)
-		)
-	)
-	(wire
-		(pts
 			(xy 260.35 57.15) (xy 260.35 60.96)
 		)
@@
 	(wire
 		(pts
-			(xy 166.37 66.04) (xy 163.83 66.04)
-		)
-		(stroke
-			(width 0)
-			(type default)
-		)
-	)
-	(wire
-		(pts
 			(xy 262.89 60.96) (xy 260.35 60.96)
 		)
@@
 	(wire
 		(pts
-			(xy 163.83 66.04) (xy 161.29 66.04)
+			(xy 161.29 66.04) (xy 166.37 66.04)
 		)
 		(stroke
@@
 	)
 	(symbol
-		(lib_id "Connector:TestPoint_Small")
-		(at 163.83 64.77 270)
-		(mirror x)
-		(unit 1)
-		(body_style 1)
-		(exclude_from_sim no)
-		(in_bom yes)
-		(on_board yes)
-		(in_pos_files yes)
-		(dnp no)
-		(property "Reference" "TP6"
-			(at 163.83 59.69 90)
-			(show_name no)
-			(do_not_autoplace no)
-			(effects
-				(font
-					(size 1.27 1.27)
-				)
-			)
-		)
-		(property "Value" "TP_CHARGER_IN"
-			(at 163.83 62.23 90)
-			(show_name no)
-			(do_not_autoplace no)
-			(effects
-				(font
-					(size 1.27 1.27)
-				)
-			)
-		)
-		(property "Footprint" "TestPoint:TestPoint_Pad_D1.0mm"
-			(at 163.83 59.69 0)
-			(hide yes)
-			(show_name no)
-			(do_not_autoplace no)
-			(effects
-				(font
-					(size 1.27 1.27)
-				)
-			)
-		)
-		(property "Datasheet" ""
-			(at 163.83 59.69 0)
-			(hide yes)
-			(show_name no)
-			(do_not_autoplace no)
-			(effects
-				(font
-					(size 1.27 1.27)
-				)
-			)
-		)
-		(property "Description" "test point"
-			(at 163.83 64.77 0)
-			(hide yes)
-			(show_name no)
-			(do_not_autoplace no)
-			(effects
-				(font
-					(size 1.27 1.27)
-				)
-			)
-		)
-		(pin "1"
-		)
-		(instances
-			(project "main_board"
-				(path "/85046142-a8d8-4f38-9e10-1de8a043d2fb"
-					(reference "TP6")
-					(unit 1)
-				)
-			)
-		)
-	)
-	(symbol
 		(lib_id "Device:R_Small")
 		(at 237.49 129.54 90)
@@
 			"386d9a97-0abb-461f-a37a-bd9f4716160b" "43456492-ceee-4855-8d5d-9fe5619975d4"
 			"4b4e7ee5-69e0-411c-9784-4df04a015421" "53a1904e-b420-4a24-8223-13aaf9ad85f0"
-			"54168efe-0095-4c93-a4db-6e33f4998587" "5535e3e1-4219-4481-9441-cfeb2b9e2c0a"
-			"5a51a076-12ab-48b1-a820-b518d063c33c" "5e0f2bb3-bbb2-4c76-8d0d-62ad4f2f65e9"
-			"64fd5779-d922-4693-96b7-b0e3da5662f5" "6c35acfa-cbdc-47be-928e-d4e991160724"
-			"6db4b4b3-7d7d-4b4c-b0a6-5804317bc59a" "6e1904c1-4656-414e-9f3f-afce59d73ad6"
-			"72d899e1-4112-4cc1-a63a-e7d48182d15d" "819a5a45-e09b-46a4-aeb7-321f80529bf6"
+			"5535e3e1-4219-4481-9441-cfeb2b9e2c0a" "5a51a076-12ab-48b1-a820-b518d063c33c"
+			"5e0f2bb3-bbb2-4c76-8d0d-62ad4f2f65e9" "64fd5779-d922-4693-96b7-b0e3da5662f5"
+			"6c35acfa-cbdc-47be-928e-d4e991160724" "6db4b4b3-7d7d-4b4c-b0a6-5804317bc59a"
+			"6e1904c1-4656-414e-9f3f-afce59d73ad6" "819a5a45-e09b-46a4-aeb7-321f80529bf6"
 			"84f46e33-2674-437a-aa40-a07343c50c38" "8f8e6347-d0c7-4d8f-81ef-4b2b457592a6"
 			"92db74ce-3153-4f7f-8562-2c0d05faa6eb" "93854cf9-6a4c-40f1-b36e-a25a84901c64"
 			"9ae6dfa6-1b81-4fbf-b74b-88b41992d5f7" "9e571e7b-3b84-4846-8b82-ef9d06d7a997"
-			"a33a5f4c-bd85-4b63-b0f7-c3cf01a27803" "a44ee3d6-54ec-48df-8d99-6b0895fb1a91"
-			"aaf31eaf-ced7-4cfb-9e3e-6cc7cdf66f11" "ae9d0504-f800-48f9-b41f-6dad09f80aad"
-			"b0048951-32d5-48b3-a81a-e7b7dc464b9a" "b0e7d2bc-5567-47d2-b0e3-d24d2aec3f8b"
+			"a44ee3d6-54ec-48df-8d99-6b0895fb1a91" "aaf31eaf-ced7-4cfb-9e3e-6cc7cdf66f11"
+			"ae9d0504-f800-48f9-b41f-6dad09f80aad" "b0e7d2bc-5567-47d2-b0e3-d24d2aec3f8b"
 			"b8fe9021-575f-4e84-928b-7c207ea4ba68" "be04fb32-50aa-486b-99da-5feceadfd928"
 			"ca51867c-a114-49f7-a05f-3abd1f64d918" "d116d68b-02a0-419b-af4c-d373d297ec5a"

Commit message: hw v0.5
Parts:
- J6: footprint Connector_USB:USB_C_Receptacle_GCT_USB4105-xx-A_16P_TopMnt_Horizontal -> Connector_USB:USB_C_Receptacle_HRO_TYPE-C-31-M-12
Changed lines of the file:
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@@
 			)
 		)
-		(property "Footprint" "Connector_USB:USB_C_Receptacle_GCT_USB4105-xx-A_16P_TopMnt_Horizontal"
+		(property "Footprint" "Connector_USB:USB_C_Receptacle_HRO_TYPE-C-31-M-12"
 			(at 39.37 53.34 0)
 			(hide yes)

Commit message: hw v1 add sw
Parts:
- added J1: power swith, Connector_JST:JST_XH_B2B-XH-A_1x02_P2.50mm_Vertical, symbol Connector_Generic:Conn_01x02
- TP7: value TP_BAT_SYSTEM -> TP_BAT_SW
Connections:
- net BAT_SYSTEM: now also J1.2 (Pin_2); no longer C22.1, IC5.9 (BAT), R19.1, R21.1, TP7.1
- new net BAT_SW: C22.1, IC5.9 (BAT), J1.1 (Pin_1), R19.1, R21.1, TP7.1
