File: hardware/main_board/main_board.kicad_sch (KiCad schematic)
At the start: 38 parts, among them IC1 E22-900M22S, IC2 INA226AIDGST, IC3 INA226AIDGST, J2 I2C External Modules, J4 WI-FI switch, U1 ESP32-C3-WROOM-02, U2 DS3231SN, U3 FM24CL16B, U5 PCA9536DR

Commit message: hw v1 cleanup
Connections:
- net BAT_SYSTEM renamed BAT_SW
Other:
- note added: "footprint DS3231M сумісний із DS3231SN"
- note removed: "footprint DS3231M, він сумісний із DS3231SN"
Changed lines of the file:
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@@
 	(text "address: 0x44"
 		(exclude_from_sim no)
-		(at 212.598 44.704 0)
+		(at 196.85 54.102 0)
 		(effects
 			(font
@@
 	(text "address: 0x40"
 		(exclude_from_sim no)
-		(at 274.828 46.228 0)
+		(at 260.096 55.372 0)
 		(effects
 			(font
@@
 		)
 	)
-	(text "footprint DS3231M, він сумісний із DS3231SN"
+	(text "footprint DS3231M сумісний із DS3231SN"
 		(exclude_from_sim no)
 		(at 149.098 58.42 0)
@@
 		)
 	)
-	(global_label "BAT_FUSED"
+	(global_label "BAT_SW"
 		(shape input)
-		(at 176.53 31.75 180)
+		(at 176.53 36.83 180)
 		(fields_autoplaced yes)
 		(effects
@@
 		)
 		(property "Intersheetrefs" "${INTERSHEET_REFS}"
-			(at 163.2034 31.75 0)
+			(at 166.5901 36.83 0)
 			(hide yes)
 			(show_name no)
@@
 		)
 	)
-	(global_label "BT_CR2032"
+	(global_label "BAT_FUSED"
 		(shape input)
-		(at 147.32 29.21 0)
+		(at 176.53 31.75 180)
 		(fields_autoplaced yes)
 		(effects
@@
 				(size 1.27 1.27)
 			)
-			(justify left)
+			(justify right)
 		)
 		(property "Intersheetrefs" "${INTERSHEET_REFS}"
-			(at 160.8884 29.21 0)
+			(at 163.2034 31.75 0)
 			(hide yes)
 			(show_name no)
@@
 					(size 1.27 1.27)
 				)
-				(justify left)
+				(justify right)
 			)
 		)
 	)
-	(global_label "USB_D+"
+	(global_label "BT_CR2032"
 		(shape input)
-		(at 63.5 154.94 270)
+		(at 147.32 29.21 0)
 		(fields_autoplaced yes)
 		(effects
@@
 				(size 1.27 1.27)
 			)
-			(justify right)
+			(justify left)
 		)
 		(property "Intersheetrefs" "${INTERSHEET_REFS}"
-			(at 63.5 165.5452 90)
+			(at 160.8884 29.21 0)
 			(hide yes)
 			(show_name no)
@@
 					(size 1.27 1.27)
 				)
-				(justify right)
+				(justify left)
 			)
 		)
 	)
-	(global_label "BAT_SYSTEM"
+	(global_label "USB_D+"
 		(shape input)
-		(at 176.53 36.83 180)
+		(at 63.5 154.94 270)
 		(fields_autoplaced yes)
 		(effects
@@
 		)
 		(property "Intersheetrefs" "${INTERSHEET_REFS}"
-			(at 162.1754 36.83 0)
+			(at 63.5 165.5452 90)
 			(hide yes)
 			(show_name no)
@@
 	)
 	(group ""
-		(members "41087be8-1307-43c1-b754-e96493624a15" "6eea7035-4f25-4a72-a618-6bd536c5cd82"
-			"d35a39dc-54a1-4f7a-8367-cdd6aca895b0"
-		)
+		(members "41087be8-1307-43c1-b754-e96493624a15" "6eea7035-4f25-4a72-a618-6bd536c5cd82")
 	)
 	(group ""
@@
 			"13595f4c-2dbe-4409-a59b-82464d33fa12" "2b167bd5-e1bd-4197-a502-864c9a7b95aa"
 			"39b9ed67-e27f-4e18-86b5-da70755efc80" "3ff4b56b-3905-47d8-ba18-f0a2ab7a4737"
-			"4ada11c3-3a60-4087-af6a-a86667fb405f" "59c6c737-c19f-4561-83bf-fb6677f94526"
-			"6de222bc-ddaf-4cf1-9a43-9c920d38dce9" "7df4dcb2-cf00-4608-89ed-0d26f69bee5f"
-			"8b3ba311-ba6f-405a-9669-d56774b09bfd" "9617faaf-6434-4a95-8d89-d22f5108b073"
-			"969bf7c8-949e-4686-a2e2-beec35f0fc5f" "cf807277-56c8-4e20-8834-dad78cc649cc"
-			"d352f9b2-7940-4ae5-a426-046b3ecf4db6" "e4cbf31c-9497-4255-bc42-33dda2f98989"
-			"f1094a68-0f73-42db-a44d-445e356ae712" "fadc9a7b-edb4-4ec2-9615-eb0089a984be"
-			"fe75700f-cfbc-4fba-9d4b-11ffd5ce39b7"
+			"40c2dfe6-be06-4bf0-ba45-912b47b86575" "4ada11c3-3a60-4087-af6a-a86667fb405f"
+			"59c6c737-c19f-4561-83bf-fb6677f94526" "6de222bc-ddaf-4cf1-9a43-9c920d38dce9"
+			"7df4dcb2-cf00-4608-89ed-0d26f69bee5f" "8b3ba311-ba6f-405a-9669-d56774b09bfd"
+			"9617faaf-6434-4a95-8d89-d22f5108b073" "969bf7c8-949e-4686-a2e2-beec35f0fc5f"
+			"cf807277-56c8-4e20-8834-dad78cc649cc" "d352f9b2-7940-4ae5-a426-046b3ecf4db6"
+			"e4cbf31c-9497-4255-bc42-33dda2f98989" "f1094a68-0f73-42db-a44d-445e356ae712"
+			"fadc9a7b-edb4-4ec2-9615-eb0089a984be" "fe75700f-cfbc-4fba-9d4b-11ffd5ce39b7"
 		)
 	)
