File: hardware/main_board/power.kicad_sch (KiCad schematic)
At the start: 46 parts, among them IC4 TPS2121RUXT, IC5 TP5000-QFN16, J1 power swith, J3 Solar panel, J5 Battary over BMS, J6 USB4105-GF-A-060, U4 TPS631000DRLR

Commit message: hw v1 fix schema
Changed lines of the file:
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@@
 	)
 	(junction
-		(at 135.89 142.24)
-		(diameter 0)
-		(color 0 0 0 0)
-	)
-	(junction
 		(at 246.38 100.33)
 		(diameter 0)
@@
 	)
 	(junction
+		(at 146.05 142.24)
+		(diameter 0)
+		(color 0 0 0 0)
+	)
+	(junction
 		(at 58.42 93.98)
 		(diameter 0)
@@
 	(wire
 		(pts
-			(xy 140.97 142.24) (xy 154.94 142.24)
-		)
-		(stroke
-			(width 0)
-			(type default)
-		)
-	)
-	(wire
-		(pts
 			(xy 193.04 34.29) (xy 193.04 54.61)
 		)
@@
 	(wire
 		(pts
-			(xy 123.19 43.18) (xy 123.19 49.53)
+			(xy 140.97 142.24) (xy 154.94 142.24)
 		)
 		(stroke
@@
 	(wire
 		(pts
-			(xy 113.03 85.09) (xy 113.03 80.01)
+			(xy 123.19 43.18) (xy 123.19 49.53)
 		)
 		(stroke
@@
 	(wire
 		(pts
-			(xy 193.04 54.61) (xy 210.82 54.61)
+			(xy 113.03 85.09) (xy 113.03 80.01)
 		)
 		(stroke
@@
 	(wire
 		(pts
-			(xy 203.2 97.79) (xy 203.2 100.33)
+			(xy 193.04 54.61) (xy 210.82 54.61)
 		)
 		(stroke
@@
 	(wire
 		(pts
-			(xy 158.75 123.19) (xy 191.77 123.19)
+			(xy 203.2 97.79) (xy 203.2 100.33)
 		)
 		(stroke
@@
 	(wire
 		(pts
-			(xy 31.75 76.2) (xy 35.56 76.2)
+			(xy 158.75 123.19) (xy 191.77 123.19)
 		)
 		(stroke
@@
 	(wire
 		(pts
-			(xy 135.89 139.7) (xy 135.89 142.24)
+			(xy 31.75 76.2) (xy 35.56 76.2)
 		)
 		(stroke
@@
 	)
 	(symbol
-		(lib_id "power:PWR_FLAG")
-		(at 135.89 139.7 0)
-		(unit 1)
-		(body_style 1)
-		(exclude_from_sim no)
-		(in_bom yes)
-		(on_board yes)
-		(in_pos_files yes)
-		(dnp no)
-		(fields_autoplaced yes)
-		(property "Reference" "#FLG08"
-			(at 135.89 137.795 0)
-			(hide yes)
-			(show_name no)
-			(do_not_autoplace no)
-			(effects
-				(font
-					(size 1.27 1.27)
-				)
-			)
-		)
-		(property "Value" "PWR_FLAG"
-			(at 135.89 134.62 0)
-			(show_name no)
-			(do_not_autoplace no)
-			(effects
-				(font
-					(size 1.27 1.27)
-				)
-			)
-		)
-		(property "Footprint" ""
-			(at 135.89 139.7 0)
-			(hide yes)
-			(show_name no)
-			(do_not_autoplace no)
-			(effects
-				(font
-					(size 1.27 1.27)
-				)
-			)
-		)
-		(property "Datasheet" ""
-			(at 135.89 139.7 0)
-			(hide yes)
-			(show_name no)
-			(do_not_autoplace no)
-			(effects
-				(font
-					(size 1.27 1.27)
-				)
-			)
-		)
-		(property "Description" "Special symbol for telling ERC where power comes from"
-			(at 135.89 139.7 0)
-			(hide yes)
-			(show_name no)
-			(do_not_autoplace no)
-			(effects
-				(font
-					(size 1.27 1.27)
-				)
-			)
-		)
-		(pin "1"
-		)
-		(instances
-			(project "main_board"
-				(path "/85046142-a8d8-4f38-9e10-1de8a043d2fb"
-					(reference "#FLG08")
-					(unit 1)
-				)
-			)
-		)
-	)
-	(symbol
 		(lib_id "power:GND")
 		(at 227.33 80.01 0)
@@
 	)
 	(symbol
+		(lib_id "power:PWR_FLAG")
+		(at 146.05 142.24 0)
+		(unit 1)
+		(body_style 1)
+		(exclude_from_sim no)
+		(in_bom yes)
+		(on_board yes)
+		(in_pos_files yes)
+		(dnp no)
+		(fields_autoplaced yes)
+		(property "Reference" "#FLG09"
+			(at 146.05 140.335 0)
+			(hide yes)
+			(show_name no)
+			(do_not_autoplace no)
+			(effects
+				(font
+					(size 1.27 1.27)
+				)
+			)
+		)
+		(property "Value" "PWR_FLAG"
+			(at 146.05 137.16 0)
+			(show_name no)
+			(do_not_autoplace no)
+			(effects
+				(font
+					(size 1.27 1.27)
+				)
+			)
+		)
+		(property "Footprint" ""
+			(at 146.05 142.24 0)
+			(hide yes)
+			(show_name no)
+			(do_not_autoplace no)
+			(effects
+				(font
+					(size 1.27 1.27)
+				)
+			)
+		)
+		(property "Datasheet" ""
+			(at 146.05 142.24 0)
+			(hide yes)
+			(show_name no)
+			(do_not_autoplace no)
+			(effects
+				(font
+					(size 1.27 1.27)
+				)
+			)
+		)
+		(property "Description" "Special symbol for telling ERC where power comes from"
+			(at 146.05 142.24 0)
+			(hide yes)
+			(show_name no)
+			(do_not_autoplace no)
+			(effects
+				(font
+					(size 1.27 1.27)
+				)
+			)
+		)
+		(pin "1"
+		)
+		(instances
+			(project "main_board"
+				(path "/85046142-a8d8-4f38-9e10-1de8a043d2fb"
+					(reference "#FLG09")
+					(unit 1)
+				)
+			)
+		)
+	)
+	(symbol
 		(lib_id "Connector_Generic:Conn_01x02")
 		(at 34.29 93.98 0)
@@
 			"1bb8972a-72fa-4ff3-a843-b0669aa1f173" "1cca1312-97a0-457c-9b92-4b3fbd3a47f6"
 			"21b88c43-9dd0-49d8-b12f-976500069705" "21e8bd7d-03fb-4584-841e-b112026eb770"
-			"234e0044-b750-4ce6-a9c9-f2488e5ac460" "238847f6-6324-423d-adf0-8e5c53b68418"
-			"253a215a-76cd-4072-a87f-5c0cc0763a8e" "2897bde0-24c5-4ca5-98df-5b7ae8e8340a"
-			"293dbedc-25cc-4692-b025-eae82c519ca2" "2b3907e9-85e8-46a7-9543-30abf013a707"
-			"2b8711ab-c171-4cdd-b713-1dc49e6b031b" "32fea740-8fe1-42ce-bfbb-56e24063d0d3"
+			"234e0044-b750-4ce6-a9c9-f2488e5ac460" "253a215a-76cd-4072-a87f-5c0cc0763a8e"
+			"2897bde0-24c5-4ca5-98df-5b7ae8e8340a" "293dbedc-25cc-4692-b025-eae82c519ca2"
+			"2b3907e9-85e8-46a7-9543-30abf013a707" "32fea740-8fe1-42ce-bfbb-56e24063d0d3"
 			"3483fbd8-38eb-44e6-acd1-453a723bfcd1" "34a7cd3c-f7d7-4211-8ab1-43ca9a3b74eb"
 			"3a3c3ed0-c340-4c9b-87bd-6a587e771fe4" "3ae9bfaa-0ceb-422b-883d-3dbb73ab8b91"
@@
 			"3c2e3962-114e-4093-b5c0-5230e4c2b832" "3e35fdc8-6e4c-4330-954a-4e7974b56a81"
 			"3e76926e-0517-41e8-95e7-a72372856a29" "3f06444e-8c45-47d7-980a-855c9e029557"
-			"3f3ae518-854d-49d9-993d-e34cff5abbce" "4055d1f4-16fd-4662-99a2-b24bc65eb00e"
-			"43d17b5b-65b9-4f36-9c1f-a2f43274dec3" "4445992e-9739-458a-8caa-1fb9e46cb5e8"
-			"4aac472e-1794-4d23-b5fc-cd36e534d65b" "4cd94a6d-7ca4-429b-9511-a1e07ab2a1cd"
-			"4e457a33-9846-4ca2-88d7-dd3c147d213b" "4e5fb91e-3d52-47c5-bd41-93a5f23473d3"
-			"4f51702d-c351-4e9e-aae7-da884285e307" "508ce01e-19e3-469d-ad14-33bc81234ac2"
-			"530906cf-dbe6-4374-b7de-262ac380ecbf" "559cfd22-4630-467c-a227-38bd915d9b94"
-			"60d4e61c-f024-4456-82ad-6e8bdd1c6214" "613e7b74-ea0f-44e1-9d0c-6c23d70eaaf2"
-			"61886f4a-d64f-4dc1-9749-4a13145e1a66" "6bc47564-2105-44c4-8d2e-e0c4821f9338"
-			"6be32338-7e36-41ad-b3f9-500ac8466d71" "6e2b87a1-f66d-41b2-863e-c88a4809d801"
-			"6f135bd0-6443-4108-851e-1cdc7d89afe3" "747afc96-20e4-420c-adac-fd0da10fbf00"
-			"768d8a6b-8436-42bf-a7df-e70eac2a8856" "76c9d31c-f683-4cf1-aa2d-97bd2dd03048"
-			"7bff3281-1d3b-4ce9-9da7-fbb3513d895a" "7c521dd6-cfa0-4bc8-b394-b79bbabb6765"
-			"889ec5d3-9bae-4833-a2bd-b164aca7015b" "8a38e827-ed0c-47d0-8d0b-428b312352d6"
-			"8e648a43-fd42-48e3-b6af-1efe384d6401" "9cce6542-8720-42f2-b79f-fd94a9f0b09c"
-			"9db17d40-4ed6-439b-95b9-0e8746b7d8e6" "a0e5d3d8-4035-4df3-9188-3d6e4219eec4"
-			"a8060f75-81ad-4382-a79e-381c18e39651" "ab302da6-25ab-4a10-b492-2a5ada7f2464"
-			"ac46b45e-6e49-41e2-9824-ee7152146eca" "ac6dfcdc-e30c-46d2-b1e8-fc0f54a02b95"
+			"3f3ae518-854d-49d9-993d-e34cff5abbce" "43d17b5b-65b9-4f36-9c1f-a2f43274dec3"
+			"4445992e-9739-458a-8caa-1fb9e46cb5e8" "4aac472e-1794-4d23-b5fc-cd36e534d65b"
+			"4cd94a6d-7ca4-429b-9511-a1e07ab2a1cd" "4e457a33-9846-4ca2-88d7-dd3c147d213b"
+			"4e5fb91e-3d52-47c5-bd41-93a5f23473d3" "4f51702d-c351-4e9e-aae7-da884285e307"
+			"508ce01e-19e3-469d-ad14-33bc81234ac2" "530906cf-dbe6-4374-b7de-262ac380ecbf"
+			"559cfd22-4630-467c-a227-38bd915d9b94" "60d4e61c-f024-4456-82ad-6e8bdd1c6214"
+			"613e7b74-ea0f-44e1-9d0c-6c23d70eaaf2" "61886f4a-d64f-4dc1-9749-4a13145e1a66"
+			"6bc47564-2105-44c4-8d2e-e0c4821f9338" "6be32338-7e36-41ad-b3f9-500ac8466d71"
+			"6e2b87a1-f66d-41b2-863e-c88a4809d801" "6f135bd0-6443-4108-851e-1cdc7d89afe3"
+			"747afc96-20e4-420c-adac-fd0da10fbf00" "768d8a6b-8436-42bf-a7df-e70eac2a8856"
+			"76c9d31c-f683-4cf1-aa2d-97bd2dd03048" "7bff3281-1d3b-4ce9-9da7-fbb3513d895a"
+			"7c521dd6-cfa0-4bc8-b394-b79bbabb6765" "889ec5d3-9bae-4833-a2bd-b164aca7015b"
+			"8a38e827-ed0c-47d0-8d0b-428b312352d6" "8e648a43-fd42-48e3-b6af-1efe384d6401"
+			"9cce6542-8720-42f2-b79f-fd94a9f0b09c" "9db17d40-4ed6-439b-95b9-0e8746b7d8e6"
+			"a0e5d3d8-4035-4df3-9188-3d6e4219eec4" "a8060f75-81ad-4382-a79e-381c18e39651"
+			"ab302da6-25ab-4a10-b492-2a5ada7f2464" "ac46b45e-6e49-41e2-9824-ee7152146eca"
+			"ac6dfcdc-e30c-46d2-b1e8-fc0f54a02b95" "adea4f3f-f172-41fe-be4b-7ba6cec04237"
 			"b455f17b-80ae-4262-92d2-b4e2811ff082" "b5ca64e6-4f51-4e08-9a45-b5660666fbf6"
-			"b5f78ead-2b1f-4247-ab0f-b54c04e742b3" "b8cccc74-5893-4c64-9247-ea106c0fd4c5"
-			"b9ab236b-0997-496f-b20b-8fc95fda56e2" "c0f61c31-87d9-4105-a779-6a82416b29da"
-			"c324fac1-4b85-45d9-ad6a-bcb0c0c3ae2a" "c37f37d6-0d0e-45b5-ba68-09cbe94aebad"
+			"b5f78ead-2b1f-4247-ab0f-b54c04e742b3" "b9ab236b-0997-496f-b20b-8fc95fda56e2"
+			"c0f61c31-87d9-4105-a779-6a82416b29da" "c324fac1-4b85-45d9-ad6a-bcb0c0c3ae2a"
+			"c37f37d6-0d0e-45b5-ba68-09cbe94aebad" "c5ee5c1c-b98b-4a42-ad71-55efc45055d4"
 			"c986afc5-fdab-4bab-a16f-8719c78f05b8" "cc539286-81e4-4fb6-90d8-33d1e9e92fbe"
 			"cc6939db-a4bc-45df-9c80-2a425d038826" "ccefb941-52fd-40db-9526-72bff9ba321a"
 			"d0baaa49-d85f-4b3f-8579-f11520550060" "d0be3640-09f7-46d7-bccd-6de44ca99449"
 			"d16ae061-ac7f-49b0-ad44-104cfcba8751" "d7b20548-dcde-4a72-abc3-629dae918232"
-			"da27c0ad-63fd-4144-b014-5088c334eb47" "ddab9e3f-8838-432c-a59a-68af22866e86"
-			"e6cee70c-b9da-45d7-9222-4989bdd44bb3" "ea332e8b-2aa6-4d06-9a9a-eafc793075a1"
-			"f01a98c9-c504-434f-9a98-534f9e1d10b5" "f06ada37-503d-49f6-81bb-00cd6d3b8e48"
-			"f1d98eac-7c5e-4143-9bef-3ed00b77e44e" "f4fd546a-d9f6-4f90-ae92-89d127cac204"
-			"fb7f6eb0-88fe-439d-b5ff-386ec3d3925d" "fecbe64d-6e0c-47b7-b903-af26cfdd07a7"
+			"d9b75963-ec63-4e0d-98f6-7b7a265f55cb" "da27c0ad-63fd-4144-b014-5088c334eb47"
+			"ddab9e3f-8838-432c-a59a-68af22866e86" "e6cee70c-b9da-45d7-9222-4989bdd44bb3"
+			"ea332e8b-2aa6-4d06-9a9a-eafc793075a1" "f01a98c9-c504-434f-9a98-534f9e1d10b5"
+			"f06ada37-503d-49f6-81bb-00cd6d3b8e48" "f1d98eac-7c5e-4143-9bef-3ed00b77e44e"
+			"f4fd546a-d9f6-4f90-ae92-89d127cac204" "fb7f6eb0-88fe-439d-b5ff-386ec3d3925d"
+			"fecbe64d-6e0c-47b7-b903-af26cfdd07a7"
 		)
 	)

Commit message: hw v1 cleanup
Changed lines of the file:
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@@
 		)
 	)
-	(label "BAT_SW"
-		(at 137.16 142.24 0)
-		(effects
-			(font
-				(size 1.27 1.27)
-			)
-			(justify left bottom)
-		)
-	)
 	(label "BAT_RAW"
 		(at 82.55 142.24 0)
@@
 		)
 	)
-	(label "BAT_SW"
-		(at 246.38 69.85 270)
-		(effects
-			(font
-				(size 1.27 1.27)
-			)
-			(justify right bottom)
-		)
-	)
 	(label "CHARGER_IN"
 		(at 166.37 66.04 0)
@@
 		)
 	)
+	(global_label "BAT_SW"
+		(shape input)
+		(at 137.16 142.24 90)
+		(fields_autoplaced yes)
+		(effects
+			(font
+				(size 1.27 1.27)
+			)
+			(justify left)
+		)
+		(property "Intersheetrefs" "${INTERSHEET_REFS}"
+			(at 137.16 132.3001 90)
+			(hide yes)
+			(show_name no)
+			(do_not_autoplace no)
+			(effects
+				(font
+					(size 1.27 1.27)
+				)
+				(justify left)
+			)
+		)
+	)
 	(global_label "BAT_SYSTEM"
 		(shape input)
@@
 		)
 	)
+	(global_label "BAT_SW"
+		(shape input)
+		(at 246.38 69.85 270)
+		(fields_autoplaced yes)
+		(effects
+			(font
+				(size 1.27 1.27)
+			)
+			(justify right)
+		)
+		(property "Intersheetrefs" "${INTERSHEET_REFS}"
+			(at 246.38 79.7899 90)
+			(hide yes)
+			(show_name no)
+			(do_not_autoplace no)
+			(effects
+				(font
+					(size 1.27 1.27)
+				)
+				(justify right)
+			)
+		)
+	)
 	(global_label "USB_D+"
 		(shape input)
@@
 			"3a5b7327-29ea-46c4-b188-dade3a891d05" "446bca8f-1785-4338-90a4-3acbc56d079e"
 			"45df5df0-49a7-48b5-8c9b-306ceffb89a3" "4b5a2695-8134-4938-a1a4-f65476441995"
-			"4fa536b8-2756-4842-ad35-6b4b9c7c7c1f" "52ea0943-58ce-4df3-a6fe-85424c5b0986"
-			"55438e4e-369c-4093-8f9a-a67cc10dd4c2" "5681f810-4cb0-40ed-bda4-6a7f29823f34"
-			"59a75b16-2ab6-41ee-9f5d-b4409d30148e" "5a83ad6b-1f05-4903-bf45-b7868b01523f"
-			"5ad97645-c2a7-4605-91a5-7f30ec024478" "5e0d8077-fdc4-41e9-843c-49fa952a939d"
-			"61c86746-630f-479b-90eb-b5edd9946112" "61fe32dc-47e5-4535-a07f-cb35cd1982ee"
-			"65385f41-4215-4b23-b21d-b5ae742e468e" "672b4037-8280-4d9b-b74b-107d9e19dd4d"
-			"67a7e8a5-5ef4-484c-99af-09eccbd90181" "6b043e90-458c-4e6e-bc3c-85f9c5c56f3a"
-			"6c5f6cf6-3dc4-452f-8594-5fad6ef657c1" "6df6c2e3-4f63-4b96-a263-3a0bf3d6c39c"
-			"6ec73630-23f6-4ac9-ab73-50c8cb5a861c" "74296e10-9a06-4646-9209-4ab08f62dee5"
-			"78fe5b25-c6cc-47c7-b7e5-edca9901703f" "7c6fa423-3135-4a56-911e-8f81a96dc4a3"
-			"7cb5467b-2f5a-4439-b26e-2d4309db3298" "7d466200-5079-477c-8ae5-74c22a0a9599"
-			"8369b098-47e4-4637-b7db-eb3d37e9ebe8" "8665b49e-96df-441b-8b34-83e4e6ed9b57"
-			"8923242e-0408-4a7a-9d36-a2f06f66726f" "8aed1963-6513-439f-9d9c-e39f5741f8f4"
-			"91383699-ee84-448a-8ec1-5efa7fa601b7" "91eacc5a-99ee-435e-80e0-4070b45dad25"
-			"91ed5a62-6bb4-47bc-be1d-354bfaea176a" "92596cd9-103e-41ad-a890-a9287c81fd9a"
-			"94e5eaae-2613-4851-9bda-9e5334aa9aa7" "98f4b1e3-6e33-41d7-91cf-de8b64d68144"
-			"9f1650aa-8443-4d0b-b19c-70c104fe2b42" "9f455579-dee3-4ed5-9e29-8b9a1bab58ac"
-			"a5d056a6-8cfe-4076-9c25-c74946f888d6" "a7d0d763-2508-4129-9bb5-0c21bd33753c"
-			"a8c3e9e8-db50-4343-a3e9-d78899da101f" "a8ed10b3-4b64-43a0-8256-74b62f06138a"
-			"ad65933a-546c-47c1-ad2e-4030bb3f2bfd" "ad6593b7-0e17-4093-8449-0796a50d651d"
-			"af27b207-8be4-45d3-9aca-13f0a328cb7e" "af6274c3-065b-4f04-8ad2-0c40b08c43e6"
-			"b3648f69-9932-4413-9221-e9bdb86ebc76" "b551ec8e-dad2-4558-a755-17559be2be69"
-			"ba4acbc7-4d3e-4f73-b9b5-9517b435303d" "bcef43e9-7ddd-403b-8944-2bd16b0f37f6"
-			"c21a18bc-a44c-4564-ad6f-a28fd276f515" "c4fa49eb-d09e-4b91-869a-f89c764a2f73"
-			"c994fc13-3e17-4af3-b290-67fa9a64b88b" "cd1324c8-9c32-4c6e-b8c5-d4187c600809"
-			"cdf9dc71-3bf7-4db8-8b77-91b71b69f0db" "ceffcbc0-2eac-4f07-ac42-2b86ec49927b"
-			"cf462874-876b-465e-8757-98dc1fd29372" "d2042bc7-0ccd-4d2c-aeba-4b931af7b949"
-			"d23d7d56-cbf1-4692-816f-0bd7abc3b27a" "d45f4f3d-72e2-4410-a75c-d62c9e4247bc"
-			"d9b8e46b-c538-4aa0-84f3-5b951262e887" "dda85249-cb80-41df-b3ce-87737a6edc5e"
-			"e59a5e53-6000-4424-aca1-6265af3cb36c" "f0cda75c-5af6-4635-8915-b140887e5891"
+			"52ea0943-58ce-4df3-a6fe-85424c5b0986" "55438e4e-369c-4093-8f9a-a67cc10dd4c2"
+			"5681f810-4cb0-40ed-bda4-6a7f29823f34" "59a75b16-2ab6-41ee-9f5d-b4409d30148e"
+			"5a83ad6b-1f05-4903-bf45-b7868b01523f" "5ad97645-c2a7-4605-91a5-7f30ec024478"
+			"5e0d8077-fdc4-41e9-843c-49fa952a939d" "61c86746-630f-479b-90eb-b5edd9946112"
+			"61fe32dc-47e5-4535-a07f-cb35cd1982ee" "65385f41-4215-4b23-b21d-b5ae742e468e"
+			"672b4037-8280-4d9b-b74b-107d9e19dd4d" "67a7e8a5-5ef4-484c-99af-09eccbd90181"
+			"6b043e90-458c-4e6e-bc3c-85f9c5c56f3a" "6c5f6cf6-3dc4-452f-8594-5fad6ef657c1"
+			"6df6c2e3-4f63-4b96-a263-3a0bf3d6c39c" "6ec73630-23f6-4ac9-ab73-50c8cb5a861c"
+			"74296e10-9a06-4646-9209-4ab08f62dee5" "78fe5b25-c6cc-47c7-b7e5-edca9901703f"
+			"7c6fa423-3135-4a56-911e-8f81a96dc4a3" "7cb5467b-2f5a-4439-b26e-2d4309db3298"
+			"7d466200-5079-477c-8ae5-74c22a0a9599" "8369b098-47e4-4637-b7db-eb3d37e9ebe8"
+			"8665b49e-96df-441b-8b34-83e4e6ed9b57" "8923242e-0408-4a7a-9d36-a2f06f66726f"
+			"8aed1963-6513-439f-9d9c-e39f5741f8f4" "91383699-ee84-448a-8ec1-5efa7fa601b7"
+			"91eacc5a-99ee-435e-80e0-4070b45dad25" "91ed5a62-6bb4-47bc-be1d-354bfaea176a"
+			"92596cd9-103e-41ad-a890-a9287c81fd9a" "94e5eaae-2613-4851-9bda-9e5334aa9aa7"
+			"98f4b1e3-6e33-41d7-91cf-de8b64d68144" "9f1650aa-8443-4d0b-b19c-70c104fe2b42"
+			"9f455579-dee3-4ed5-9e29-8b9a1bab58ac" "a5d056a6-8cfe-4076-9c25-c74946f888d6"
+			"a7d0d763-2508-4129-9bb5-0c21bd33753c" "a8c3e9e8-db50-4343-a3e9-d78899da101f"
+			"a8ed10b3-4b64-43a0-8256-74b62f06138a" "ad65933a-546c-47c1-ad2e-4030bb3f2bfd"
+			"ad6593b7-0e17-4093-8449-0796a50d651d" "af27b207-8be4-45d3-9aca-13f0a328cb7e"
+			"af6274c3-065b-4f04-8ad2-0c40b08c43e6" "b3648f69-9932-4413-9221-e9bdb86ebc76"
+			"b551ec8e-dad2-4558-a755-17559be2be69" "ba4acbc7-4d3e-4f73-b9b5-9517b435303d"
+			"bcef43e9-7ddd-403b-8944-2bd16b0f37f6" "c21a18bc-a44c-4564-ad6f-a28fd276f515"
+			"c4fa49eb-d09e-4b91-869a-f89c764a2f73" "c994fc13-3e17-4af3-b290-67fa9a64b88b"
+			"cd1324c8-9c32-4c6e-b8c5-d4187c600809" "cdf9dc71-3bf7-4db8-8b77-91b71b69f0db"
+			"ceffcbc0-2eac-4f07-ac42-2b86ec49927b" "cf462874-876b-465e-8757-98dc1fd29372"
+			"d2042bc7-0ccd-4d2c-aeba-4b931af7b949" "d23d7d56-cbf1-4692-816f-0bd7abc3b27a"
+			"d45f4f3d-72e2-4410-a75c-d62c9e4247bc" "d9b8e46b-c538-4aa0-84f3-5b951262e887"
+			"dda85249-cb80-41df-b3ce-87737a6edc5e" "e59a5e53-6000-4424-aca1-6265af3cb36c"
+			"ea40929e-bf3d-461f-94e1-153f77da3d61" "f0cda75c-5af6-4635-8915-b140887e5891"
 			"f495309c-d747-46c3-8494-02edf0a11d40" "f536d72d-80f3-4853-9db0-dcf755de0d07"
 			"f7136697-fd5a-42c2-8ba9-51beae0a2d87" "f77fd21c-bb1b-47e1-9d84-d0d9f610e0a3"
@@
 			"1107b461-7615-4e30-bdd4-ec4bc6acc95c" "15c3fdea-2707-4d32-98f5-c11898006989"
 			"16a8fed1-dd3b-4e04-9203-64f9bebfa68e" "17a14a58-51e4-442e-a53b-d007ed534f12"
-			"1bb8972a-72fa-4ff3-a843-b0669aa1f173" "1cca1312-97a0-457c-9b92-4b3fbd3a47f6"
-			"21b88c43-9dd0-49d8-b12f-976500069705" "21e8bd7d-03fb-4584-841e-b112026eb770"
-			"234e0044-b750-4ce6-a9c9-f2488e5ac460" "253a215a-76cd-4072-a87f-5c0cc0763a8e"
-			"2897bde0-24c5-4ca5-98df-5b7ae8e8340a" "293dbedc-25cc-4692-b025-eae82c519ca2"
-			"2b3907e9-85e8-46a7-9543-30abf013a707" "32fea740-8fe1-42ce-bfbb-56e24063d0d3"
-			"3483fbd8-38eb-44e6-acd1-453a723bfcd1" "34a7cd3c-f7d7-4211-8ab1-43ca9a3b74eb"
-			"3a3c3ed0-c340-4c9b-87bd-6a587e771fe4" "3ae9bfaa-0ceb-422b-883d-3dbb73ab8b91"
-			"3afb402a-f1d5-44a6-af27-ba3e81f12eec" "3c0c4c3e-b9bd-4bfe-a140-1596e5be1725"
-			"3c2e3962-114e-4093-b5c0-5230e4c2b832" "3e35fdc8-6e4c-4330-954a-4e7974b56a81"
+			"18ef5681-a9c7-4f3d-a161-b51e13bc7c9d" "1bb8972a-72fa-4ff3-a843-b0669aa1f173"
+			"1cca1312-97a0-457c-9b92-4b3fbd3a47f6" "21b88c43-9dd0-49d8-b12f-976500069705"
+			"21e8bd7d-03fb-4584-841e-b112026eb770" "234e0044-b750-4ce6-a9c9-f2488e5ac460"
+			"253a215a-76cd-4072-a87f-5c0cc0763a8e" "2897bde0-24c5-4ca5-98df-5b7ae8e8340a"
+			"293dbedc-25cc-4692-b025-eae82c519ca2" "2b3907e9-85e8-46a7-9543-30abf013a707"
+			"32fea740-8fe1-42ce-bfbb-56e24063d0d3" "3483fbd8-38eb-44e6-acd1-453a723bfcd1"
+			"34a7cd3c-f7d7-4211-8ab1-43ca9a3b74eb" "3a3c3ed0-c340-4c9b-87bd-6a587e771fe4"
+			"3ae9bfaa-0ceb-422b-883d-3dbb73ab8b91" "3afb402a-f1d5-44a6-af27-ba3e81f12eec"
+			"3c0c4c3e-b9bd-4bfe-a140-1596e5be1725" "3c2e3962-114e-4093-b5c0-5230e4c2b832"
 			"3e76926e-0517-41e8-95e7-a72372856a29" "3f06444e-8c45-47d7-980a-855c9e029557"
 			"3f3ae518-854d-49d9-993d-e34cff5abbce" "43d17b5b-65b9-4f36-9c1f-a2f43274dec3"

Commit message: hw v1 battery selection
Parts:
- added R6: 0R, Resistor_SMD:R_0603_1608Metric, symbol Device:R_Small
- added U6: USBLC6-2SC6, Package_TO_SOT_SMD:SOT-23-6, symbol Power_Protection:USBLC6-2SC6
Connections:
- net CHARGER_IN: now also R6.1
- net GND: now also U6.2 (GND)
- net USB_5V: now also U6.5 (VBUS)
- net USB_D+: now also U6.4 (I/O2); no longer J6.A6 (D+), J6.B6 (D+)
- net USB_D-: now also U6.6 (I/O1); no longer J6.A7 (D-), J6.B7 (D-)
- net at IC5.13 (CS): now also R6.2
- new net: J6.A7 (D-), J6.B7 (D-), U6.1 (I/O1)
- new net: J6.A6 (D+), J6.B6 (D+), U6.3 (I/O2)
- no-connect marks 3 -> 2
Other:
- moved on the sheet: R23, R24

Commit message: hw v1 clean up
Changed lines of the file:
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@@
 	(global_label "BAT_SW"
 		(shape input)
-		(at 246.38 69.85 270)
+		(at 246.38 78.74 0)
 		(fields_autoplaced yes)
 		(effects
@@
 				(size 1.27 1.27)
 			)
-			(justify right)
+			(justify left)
 		)
 		(property "Intersheetrefs" "${INTERSHEET_REFS}"
-			(at 246.38 79.7899 90)
+			(at 256.3199 78.74 0)
 			(hide yes)
 			(show_name no)
@@
 					(size 1.27 1.27)
 				)
-				(justify right)
+				(justify left)
 			)
 		)
@@
 	)
 	(group ""
-		(members "0283645c-0d63-4466-83ee-c85f18f6a814" "02b8abf7-262b-45ed-b5a9-8ffd74ec4ca8"
-			"0c4faf9c-3f1d-413b-8199-21afcd58c5a1" "0c9404a3-5f46-42fc-acfc-fe43d5502356"
-			"16791b80-4310-4679-a653-713a5f871865" "16d6e64c-bc85-4f88-a462-e342cf65f542"
-			"287301f7-4408-40eb-bd0e-1daceda72c99" "43f1dc2d-1e48-4526-97ef-8bd3942bdf46"
-			"4516696e-8949-4934-9b2b-eba526f2d694" "45e089ea-4381-4494-8bc1-3d1da541cd68"
-			"4eacd1ab-c2b6-4043-a634-e4a58da0d341" "51bb489e-e8a8-49cd-a8e7-a9345a9200ad"
-			"52106639-2a39-49f1-8a47-e0c0fd456385" "5b593a41-89c6-4aeb-b041-820372c1202d"
-			"5c45ed09-d3ca-48cc-8ed9-2df6bf48f834" "5e55a116-cd81-49c2-8057-99740a1226c7"
-			"65335205-e933-4e0a-afa8-73bdd648b47d" "7ad1244b-af3f-46ec-b037-68e506e111c5"
-			"7d029e2d-b397-48ed-9555-6c4915abcc62" "833b1397-1a68-4bc1-918b-eaa461af7540"
-			"8f9ba718-0e35-49ab-96e6-903bd0c3bb2f" "9376be83-3ea7-4fff-91b3-286bdf7c5e7f"
-			"9d2a2355-1c52-4d65-aa7f-db2d17af42b1" "a42a7972-71ac-45e0-87dd-2bda3120e621"
-			"a52da568-b73c-4486-a088-b8a2fa53ae0c" "a531fb23-b070-4b73-8ef4-8724b90e19bc"
-			"a6e17dea-066a-41c2-b77f-7daf086aa744" "ab22102d-e6db-47e7-ac48-21a4cef85b6d"
-			"b10e90f4-b758-4373-82aa-dc0d04461a07" "b756311c-813c-4aed-ac3a-2ace6525fc32"
-			"b799c260-937f-4f69-98a6-d5506f92b733" "bc2696f4-8189-4b58-bca8-9a41aa3f2e85"
-			"bfeff36c-afad-4c74-8490-04d3f597559c" "c2d93274-8fea-4bde-ba8b-fd2f2410daec"
-			"c349449d-3681-4cf8-b63b-aed959f3efa6" "c63d0da7-42ad-4ae8-a2f8-2ca94def4a58"
-			"c7e5f2d0-5882-4ecb-b06f-91100750ae06" "caeacd33-f18d-42da-801c-434db62e8372"
-			"cb924b70-020c-45ef-9678-e31d56df6c1f" "d281928a-0a04-43c3-a18b-b82729c25f27"
-			"dcd6c2ab-bcde-4468-8cbd-c3098a539139" "e9717762-436e-4f4d-bbf5-9a71a2e10967"
-			"ec88d59c-4287-46b3-9420-9784dbc32961" "f245171e-f67f-4843-91d4-dea5f6870e39"
-		)
-	)
-	(group ""

Commit message: software
Parts:
- added F2: 0ZCK0075FF2E, Fuse:Fuse_0805_2012Metric, symbol Device:Polyfuse_Small
- added F3: 0ZCH0075AF2E, Fuse:Fuse_1210_3225Metric, symbol Device:Polyfuse_Small
- added R29: 0R, Resistor_SMD:R_0603_1608Metric, symbol Device:R_Small
- R15: value 100mR -> 20mR
Connections:
- net +3V3: now also R29.2; no longer C14.1, C16.1, R22.1, TP8.1, U4.1 (VOUT)
- net SOLAR+: now also F3.2; no longer J3.1 (Pin_1)
- net USB_5V: now also F2.2; no longer J6.A4 (VBUS), J6.A9 (VBUS), J6.B4 (VBUS), J6.B9 (VBUS)
- new net: C14.1, C16.1, R22.1, R29.1, TP8.1, U4.1 (VOUT)
- new net: F3.1, J3.1 (Pin_1)
- new net: F2.1, J6.A4 (VBUS), J6.A9 (VBUS), J6.B4 (VBUS), J6.B9 (VBUS)
Other:
- moved on the sheet: R15, TP1, TP5
