File: hardware/sensor_board/sensor_board.kicad_sch (KiCad schematic)
At the start: 3 parts, among them J1 I2C Connector, U1 CJMCU-3935, U2 BME280

Commit message: hw v1 battery selection
Parts:
- added C1, C2: 100nf, Capacitor_THT:C_Disc_D5.0mm_W2.5mm_P2.50mm, symbol Device:C_Small
Connections:
- net +3V3: now also J1.2 (Pin_2), C1.2, C2.2; no longer J1.1 (Pin_1)
- net GND: now also J1.1 (Pin_1), C1.1, C2.1; no longer J1.2 (Pin_2)
